Commit message: fixes for the models

File: robots/puddles.xacro (robot description, xacro)
@@ -5,7 +5,7 @@
   <xacro:arg name="inertial_reference_frame" default="world"/>
   <!-- Include the Robot macro file -->
-  <xacro:include filename="$(find riptide_descriptions)/urdf/robot_base.xacro"/>
+  <xacro:include filename="$(find riptide_descriptions2)/urdf/robot_base.xacro"/>
   <!-- Read the config -->
-  <xacro:property name="yaml_file" value="$(find riptide_descriptions)/config/puddles.yaml" />
+  <xacro:property name="yaml_file" value="$(find riptide_descriptions2)/config/puddles.yaml" />
   <xacro:property name="config" value="${load_yaml(yaml_file)}"/>
   <!-- Create robot -->

File: robots/tempest.xacro (robot description, xacro)
@@ -5,7 +5,7 @@
   <xacro:arg name="inertial_reference_frame" default="world"/>
   <!-- Include the Robot macro file -->
-  <xacro:include filename="$(find riptide_descriptions)/urdf/robot_base.xacro"/>
+  <xacro:include filename="$(find riptide_descriptions2)/urdf/robot_base.xacro"/>
   <!-- Read the config -->
-  <xacro:property name="yaml_file" value="$(find riptide_descriptions)/config/tempest.yaml" />
+  <xacro:property name="yaml_file" value="$(find riptide_descriptions2)/config/tempest.yaml" />
   <xacro:property name="config" value="${load_yaml(yaml_file)}"/>
   <!-- Create robot -->

File: urdf/snippets.xacro (robot description, xacro)
@@ -129,5 +129,5 @@
         </xacro:camera_macro>
         <!-- Right camera -->
-        <xacro:camera_macro namespace="${namespace}" name="${name}_right" parent_link="${camera_namespace}/left_link" update_rate="${update_rate}" hfov="${hfov}" width="${width}" height="${height}" stddev="${stddev}" baseline="${baseline}">
+        <xacro:camera_macro namespace="${namespace}" name="${name}_right" parent_link="${camera_namespace}_left_link" update_rate="${update_rate}" hfov="${hfov}" width="${width}" height="${height}" stddev="${stddev}" baseline="${baseline}">
             <origin xyz="0 ${-baseline} 0" />
         </xacro:camera_macro>

Commit message: beat the xacro into working shape

File: robots/puddles.xacro (robot description, xacro)
@@ -9,4 +9,6 @@
   <xacro:property name="yaml_file" value="$(find riptide_descriptions2)/config/puddles.yaml" />
   <xacro:property name="config" value="${load_yaml(yaml_file)}"/>
+  <xacro:property name="body_file" value="$(find riptide_descriptions2)/meshes/Puddles.dae"/>
+  <xacro:property name="prop_file" value="$(find riptide_descriptions2)/meshes/Propeller.dae"/>
   <!-- Create robot -->
   <xacro:robot_base

File: robots/tempest.xacro (robot description, xacro)
@@ -9,4 +9,6 @@
   <xacro:property name="yaml_file" value="$(find riptide_descriptions2)/config/tempest.yaml" />
   <xacro:property name="config" value="${load_yaml(yaml_file)}"/>
+  <xacro:property name="body_file" value="$(find riptide_descriptions2)/meshes/Tempest.dae"/>
+  <xacro:property name="prop_file" value="$(find riptide_descriptions2)/meshes/Propeller.dae"/>
   <!-- Create robot -->
   <xacro:robot_base

File: urdf/robot_actuators.xacro (robot description, xacro)
@@ -20,5 +20,5 @@
         namespace="${namespace}"
         thruster_id="${index}"
-        mesh_filename="${config['mesh']}"
+        mesh_filename="${prop_file}"
         rotor_constant="${config['rotor_constant']}">
         <origin xyz="${thruster['pose'][0]} ${thruster['pose'][1]} ${thruster['pose'][2]}"

File: urdf/robot_base.xacro (robot description, xacro)
@@ -13,10 +13,10 @@
       <visual>
         <geometry>
-          <mesh filename="${config['mesh']}" scale="1 1 1"/>
+          <mesh filename="${body_file}" scale="1 1 1"/>
         </geometry>
       </visual>
       <collision>
         <geometry>
-          <mesh filename="${config['mesh']}" scale="1 1 1"/>
+          <mesh filename="${body_file}" scale="1 1 1"/>
         </geometry>
       </collision>

File: urdf/robot_sensors.xacro (robot description, xacro)
@@ -49,5 +49,5 @@
       imu_suffix=""
       parent_link="${namespace}/origin"
-      imu_topic="${imu['topic']}"
+      imu_topic="${namespace}/${imu['topic']}"
       gyroscope_noise_density="0.0003394"
       gyroscope_random_walk="0.000038785"

File: urdf/snippets.xacro (robot description, xacro)
@@ -77,26 +77,18 @@
                         <stddev>${stddev}</stddev>
                     </noise>
-                    <!-- <distortion>
-                <k1>${k1l}</k1>
-                <k2>${k2l}</k2>
-                <k3>${k3l}</k3>
-                <p1>${p1l}</p1>
-                <p2>${p2l}</p2>
-                <center>0.5 0.5</center>
-              </distortion> -->
                 </camera>
                 <plugin name="${name}_controller" filename="libgazebo_ros_camera.so">
                     <alwaysOn>true</alwaysOn>
-                    <updateRate>${update_rate}</updateRate>
-                    <cameraName>${name}</cameraName>
-                    <imageTopicName>image_raw</imageTopicName>
-                    <cameraInfoTopicName>camera_info</cameraInfoTopicName>
+                    <ros>
+                        <!-- topics need to be prefixed with camera_name for remapping -->
+                        <camera_name>${name}</camera_name>
+                        <remapping>${name}/image_raw:=${namespace}/${name}/image_raw</remapping>
+                        <remapping>${name}/image_raw/compressed:=${namespace}/${name}/image_raw/compressed</remapping>
+                        <remapping>${name}/camera_info:=${namespace}/${name}/camera_info</remapping>
+                    </ros>
+                    <!--<imageTopicName>image_raw</imageTopicName>
+                    <cameraInfoTopicName>camera_info</cameraInfoTopicName>-->
                     <frameName>${namespace}/${name}_optical</frameName>
                     <hackBaseline>${baseline}</hackBaseline>
-                    <!-- <distortionK1>${k1l}</distortionK1>
-              <distortionK2>${k2l}</distortionK2>
-              <distortionK3>${k3l}</distortionK3>
-              <distortionT1>${p1l}</distortionT1>
-              <distortionT2>${p2l}</distortionT2> -->
                 </plugin>
                 <always_on>1</always_on>
@@ -106,8 +98,8 @@
     </xacro:macro>
     <xacro:macro name="stereo_macro" params="namespace parent_link name update_rate hfov width height stddev baseline *origin">
-        <xacro:camera_macro namespace="${namespace}" name="${name}_left" parent_link="${parent_link}" update_rate="${update_rate}" hfov="${hfov}" width="${width}" height="${height}" stddev="${stddev}" baseline="${baseline}">
+        <xacro:camera_macro namespace="${namespace}/${name}" name="left" parent_link="${parent_link}" update_rate="${update_rate}" hfov="${hfov}" width="${width}" height="${height}" stddev="${stddev}" baseline="${baseline}">
             <xacro:insert_block name="origin" />
         </xacro:camera_macro>
-        <xacro:camera_macro namespace="${namespace}" name="${name}_right" parent_link="${namespace}/${name}/left_link" update_rate="${update_rate}" hfov="${hfov}" width="${width}" height="${height}" stddev="${stddev}" baseline="${baseline}">
+        <xacro:camera_macro namespace="${namespace}" name="right" parent_link="${namespace}/${name}/left_link" update_rate="${update_rate}" hfov="${hfov}" width="${width}" height="${height}" stddev="${stddev}" baseline="${baseline}">
             <origin xyz="0 ${-baseline} 0" />
         </xacro:camera_macro>
@@ -125,9 +117,9 @@
             <child link="${camera_namespace}/base_link" />
         </joint>
-        <xacro:camera_macro namespace="${namespace}" name="${name}_left" parent_link="${camera_namespace}/base_link" update_rate="${update_rate}" hfov="${hfov}" width="${width}" height="${height}" stddev="${stddev}" baseline="${baseline}">
+        <xacro:camera_macro namespace="${namespace}/${name}" name="left" parent_link="${camera_namespace}/base_link" update_rate="${update_rate}" hfov="${hfov}" width="${width}" height="${height}" stddev="${stddev}" baseline="${baseline}">
             <origin xyz="0 0 0" />
         </xacro:camera_macro>
         <!-- Right camera -->
-        <xacro:camera_macro namespace="${namespace}" name="${name}_right" parent_link="${camera_namespace}_left_link" update_rate="${update_rate}" hfov="${hfov}" width="${width}" height="${height}" stddev="${stddev}" baseline="${baseline}">
+        <xacro:camera_macro namespace="${namespace}/${name}" name="right" parent_link="${camera_namespace}/left_link" update_rate="${update_rate}" hfov="${hfov}" width="${width}" height="${height}" stddev="${stddev}" baseline="${baseline}">
             <origin xyz="0 ${-baseline} 0" />
         </xacro:camera_macro>
@@ -178,5 +170,5 @@
                     </range>
                 </ray>
-                <plugin filename="libgazebo_ros_range.so" name="dvl${suffix}_sonar${index}">
+                <plugin filename="libgazebo_ros_ray_sensor.so" name="dvl${suffix}_sonar${index}">
                     <gaussianNoise>0.005</gaussianNoise>
                     <alwaysOn>true</alwaysOn>
@@ -185,5 +177,6 @@
                     <frameName>${namespace}/dvl${suffix}_sonar${index}_link</frameName>
                     <fov>0.06</fov>
-                    <radiation>ultrasound</radiation>
+                    <radiation_type>ultrasound</radiation_type>
+                    <output_type>sensor_msgs/Range</output_type>
                 </plugin>
             </sensor>
