Commit message: Changed to tempest

File: robots/tempest.xacro (robot description, xacro)
@@ -1,11 +1,11 @@
 <?xml version="1.0"?>
-<robot name="titan" xmlns:xacro="http://www.ros.org/wiki/xacro" >
+<robot name="tempest" xmlns:xacro="http://www.ros.org/wiki/xacro" >
   <xacro:arg name="debug" default="0"/>
-  <xacro:arg name="namespace" default="titan"/>
+  <xacro:arg name="namespace" default="tempest"/>
   <xacro:arg name="inertial_reference_frame" default="world"/>
   <!-- Include the Robot macro file -->
   <xacro:include filename="$(find riptide_descriptions)/urdf/robot_base.xacro"/>
   <!-- Read the config -->
-  <xacro:property name="yaml_file" value="$(find riptide_descriptions)/config/titan.yaml" />
+  <xacro:property name="yaml_file" value="$(find riptide_descriptions)/config/tempest.yaml" />
   <xacro:property name="config" value="${load_yaml(yaml_file)}"/>
   <!-- Create robot -->

Commit message: Fix mesh path for rviz

File: robots/tempest.xacro (robot description, xacro)
@@ -9,6 +9,6 @@
   <xacro:property name="yaml_file" value="$(find riptide_descriptions2)/config/tempest.yaml" />
   <xacro:property name="config" value="${load_yaml(yaml_file)}"/>
-  <xacro:property name="body_file" value="$(find riptide_descriptions2)/meshes/Tempest.dae"/>
-  <xacro:property name="prop_file" value="$(find riptide_descriptions2)/meshes/Propeller.dae"/>
+  <xacro:property name="body_file" value="package://riptide_descriptions2/meshes/Tempest.dae"/>
+  <xacro:property name="prop_file" value="package://riptide_descriptions2/meshes/Propeller.dae"/>
   <!-- Create robot -->
   <xacro:robot_base
