Commit message: added some props, puddles visual mesh nicer

File: urdf/robot_base.xacro (robot description, xacro)
@@ -13,5 +13,5 @@
       <visual>
         <geometry>
-          <mesh filename="${config['mesh']}" scale="1 1 1"/>
+          <mesh filename="${config['visual_mesh']}" scale="1 1 1"/>
         </geometry>
       </visual>

Commit message: fixing package versions

File: urdf/robot_base.xacro (robot description, xacro)
@@ -2,6 +2,6 @@
 <!-- All coordinates in file must follow ROS conventions: x forward, z up -->
 <robot xmlns:xacro="http://www.ros.org/wiki/xacro" >
-  <xacro:include filename="$(find riptide_descriptions)/urdf/snippets.xacro" />
-  <xacro:include filename="$(find riptide_descriptions)/urdf/robot.gazebo.xacro" />
+  <xacro:include filename="$(find riptide_descriptions2)/urdf/snippets.xacro" />
+  <xacro:include filename="$(find riptide_descriptions2)/urdf/robot.gazebo.xacro" />
   <xacro:macro name="robot_base"
     params="namespace config inertial_reference_frame">
@@ -50,6 +50,6 @@
       </plugin>
     </gazebo>
-    <xacro:include filename="$(find riptide_descriptions)/urdf/robot_sensors.xacro" />
-    <xacro:include filename="$(find riptide_descriptions)/urdf/robot_actuators.xacro" />
+    <xacro:include filename="$(find riptide_descriptions2)/urdf/robot_sensors.xacro" />
+    <xacro:include filename="$(find riptide_descriptions2)/urdf/robot_actuators.xacro" />
   </xacro:macro>
 </robot>

File: urdf/snippets.xacro (robot description, xacro)
@@ -1,81 +1,81 @@
 <?xml version="1.0"?>
-<robot xmlns:xacro="http://www.ros.org/wiki/xacro" >
-  <!-- Makes a blank inertia (gazebo needs this sometimes) -->
-  <xacro:macro name="dummy_inertia">
-    <inertial>
-      <mass value="0.00001" />
-      <inertia ixx="0.000001" ixy="0.0" ixz="0.0" iyy="0.000001" iyz="0.0" izz="0.000001" />
-    </inertial>
-  </xacro:macro>
-  <xacro:macro name="no_collision">
-    <collision>
-      <geometry>
-        <cylinder length="${0.000001}" radius="${0.000001}" />
-      </geometry>
-      <origin xyz="0 0 0" rpy="0 ${0.5*pi} 0"/>
-    </collision>
-  </xacro:macro>
-  <!-- Ground truth position -->
-  <xacro:macro name="default_pose_3d_macro" params="namespace parent_link inertial_reference_frame">
-    <!-- Mount a 3D pose sensor -->
-    <link name="${namespace}/pose_sensor_link">
-      <xacro:dummy_inertia />
-    </link>
-    <joint name="${namespace}/pose_sensor_joint" type="revolute">
-      <axis xyz="0 0 1"/>
-      <parent link="${parent_link}"/>
-      <child link="${namespace}/pose_sensor_link"/>
-      <limit effort="0" lower="0" upper="0" velocity="0"/>
-    </joint>
-    <gazebo>
-      <plugin name="pose_3d_plugin" filename="libuuv_gazebo_ros_pose_gt_plugin.so">
-        <robot_namespace>${namespace}</robot_namespace>
-        <link_name>${namespace}/base_link</link_name>
-        <sensor_topic>pose_gt</sensor_topic>
-        <static_reference_frame>${inertial_reference_frame}</static_reference_frame>
-        <noise_sigma>0</noise_sigma>
-        <noise_amplitude>0</noise_amplitude>
-        <update_rate>20</update_rate>
-        <enable_gazebo_messages>false</enable_gazebo_messages>
-        <publish_ned_odom>false</publish_ned_odom>
-      </plugin>
-    </gazebo>
-  </xacro:macro>
-  <!-- TODO: Add camera distortion -->
-  <xacro:macro name="camera_macro" params="namespace name parent_link update_rate hfov width height stddev baseline:=0 *origin">
-    <link name="${namespace}/${name}_link">
-        <xacro:dummy_inertia />
-        <xacro:no_collision />
-    </link>
-    <joint name="${namespace}/${name}_joint" type="fixed">
-        <xacro:insert_block name="origin" />
-        <parent link="${parent_link}" />
-        <child link="${namespace}/${name}_link" />
-    </joint>
-    <link name="${namespace}/${name}_optical" />
-    <joint name="${namespace}/${name}_optical_joint" type="fixed">
-      <parent link="${namespace}/${name}_link" />
-      <child link="${namespace}/${name}_optical" />
-      <origin rpy="${-pi/2} 0 ${-pi/2}"></origin>
-    </joint>
-    <gazebo reference="${namespace}/${name}_link">
-        <sensor name="${name}" type="camera">
-          <camera>
-              <horizontal_fov>${hfov}</horizontal_fov>
-              <image>
-                <width>${width}</width>
-                <height>${height}</height>
-                <format>R8G8B8</format>
-              </image>
-              <clip>
-                <near>0.05</near>
-                <far>3000</far>
-              </clip>
-              <noise>
-                <type>gaussian</type>
-                <mean>0.0</mean>
-                <stddev>${stddev}</stddev>
-              </noise>
-              <!-- <distortion>
+<robot xmlns:xacro="http://www.ros.org/wiki/xacro">
+    <!-- Makes a blank inertia (gazebo needs this sometimes) -->
+    <xacro:macro name="dummy_inertia">
+        <inertial>
+            <mass value="0.00001" />
+            <inertia ixx="0.000001" ixy="0.0" ixz="0.0" iyy="0.000001" iyz="0.0" izz="0.000001" />
+        </inertial>
+    </xacro:macro>
+    <xacro:macro name="no_collision">
+        <collision>
+            <geometry>
+                <cylinder length="${0.000001}" radius="${0.000001}" />
+            </geometry>
+            <origin xyz="0 0 0" rpy="0 ${0.5*pi} 0" />
+        </collision>
+    </xacro:macro>
+    <!-- Ground truth position -->
+    <xacro:macro name="default_pose_3d_macro" params="namespace parent_link inertial_reference_frame">
+        <!-- Mount a 3D pose sensor -->
+        <link name="${namespace}/pose_sensor_link">
+            <xacro:dummy_inertia />
+        </link>
+        <joint name="${namespace}/pose_sensor_joint" type="revolute">
+            <axis xyz="0 0 1" />
+            <parent link="${parent_link}" />
+            <child link="${namespace}/pose_sensor_link" />
+            <limit effort="0" lower="0" upper="0" velocity="0" />
+        </joint>
+        <gazebo>
+            <plugin name="pose_3d_plugin" filename="libuuv_gazebo_ros_pose_gt_plugin.so">
+                <robot_namespace>${namespace}</robot_namespace>
+                <link_name>${namespace}/base_link</link_name>
+                <sensor_topic>pose_gt</sensor_topic>
+                <static_reference_frame>${inertial_reference_frame}</static_reference_frame>
+                <noise_sigma>0</noise_sigma>
+                <noise_amplitude>0</noise_amplitude>
+                <update_rate>20</update_rate>
+                <enable_gazebo_messages>false</enable_gazebo_messages>
+                <publish_ned_odom>false</publish_ned_odom>
+            </plugin>
+        </gazebo>
+    </xacro:macro>
+    <!-- TODO: Add camera distortion -->
+    <xacro:macro name="camera_macro" params="namespace name parent_link update_rate hfov width height stddev baseline:=0 *origin">
+        <link name="${namespace}/${name}_link">
+            <xacro:dummy_inertia />
+            <xacro:no_collision />
+        </link>
+        <joint name="${namespace}/${name}_joint" type="fixed">
+            <xacro:insert_block name="origin" />
+            <parent link="${parent_link}" />
+            <child link="${namespace}/${name}_link" />
+        </joint>
+        <link name="${namespace}/${name}_optical" />
+        <joint name="${namespace}/${name}_optical_joint" type="fixed">
+            <parent link="${namespace}/${name}_link" />
+            <child link="${namespace}/${name}_optical" />
+            <origin rpy="${-pi/2} 0 ${-pi/2}"></origin>
+        </joint>
+        <gazebo reference="${namespace}/${name}_link">
+            <sensor name="${name}" type="camera">
+                <camera>
+                    <horizontal_fov>${hfov}</horizontal_fov>
+                    <image>
+                        <width>${width}</width>
+                        <height>${height}</height>
+                        <format>R8G8B8</format>
+                    </image>
+                    <clip>
+                        <near>0.05</near>
+                        <far>3000</far>
+                    </clip>
+                    <noise>
+                        <type>gaussian</type>
+                        <mean>0.0</mean>
+                        <stddev>${stddev}</stddev>
+                    </noise>
+                    <!-- <distortion>
                 <k1>${k1l}</k1>
                 <k2>${k2l}</k2>
@@ -85,248 +85,181 @@
                 <center>0.5 0.5</center>
               </distortion> -->
-          </camera>
-          <plugin name="${name}_controller" filename="libgazebo_ros_camera.so">
-              <alwaysOn>true</alwaysOn>
-              <updateRate>${update_rate}</updateRate>
-              <cameraName>${name}</cameraName>
-              <imageTopicName>image_raw</imageTopicName>
-              <cameraInfoTopicName>camera_info</cameraInfoTopicName>
-              <frameName>${namespace}/${name}_optical</frameName>
-              <hackBaseline>${baseline}</hackBaseline>
-              <!-- <distortionK1>${k1l}</distortionK1>
+                </camera>
+                <plugin name="${name}_controller" filename="libgazebo_ros_camera.so">
+                    <alwaysOn>true</alwaysOn>
+                    <updateRate>${update_rate}</updateRate>
+                    <cameraName>${name}</cameraName>
+                    <imageTopicName>image_raw</imageTopicName>
+                    <cameraInfoTopicName>camera_info</cameraInfoTopicName>
+                    <frameName>${namespace}/${name}_optical</frameName>
+                    <hackBaseline>${baseline}</hackBaseline>
+                    <!-- <distortionK1>${k1l}</distortionK1>
               <distortionK2>${k2l}</distortionK2>
               <distortionK3>${k3l}</distortionK3>
               <distortionT1>${p1l}</distortionT1>
               <distortionT2>${p2l}</distortionT2> -->
-          </plugin>
-          <always_on>1</always_on>
-          <update_rate>${update_rate}</update_rate>
-        </sensor>
-    </gazebo>
-  </xacro:macro>
-  <xacro:macro name="stereo_macro" params="namespace parent_link name update_rate hfov width height stddev baseline *origin">
-    <xacro:camera_macro
-      namespace="${namespace}"
-      name="${name}/left"
-      parent_link="${parent_link}"
-      update_rate="${update_rate}"
-      hfov="${hfov}"
-      width="${width}"
-      height="${height}"
-      stddev="${stddev}"
-      baseline="${baseline}">
-      <xacro:insert_block name="origin" />
-    </xacro:camera_macro>
-    <xacro:camera_macro
-      namespace="${namespace}"
-      name="${name}/right"
-      parent_link="${namespace}/${name}/left_link"
-      update_rate="${update_rate}"
-      hfov="${hfov}"
-      width="${width}"
-      height="${height}"
-      stddev="${stddev}"
-      baseline="${baseline}">
-      <origin xyz="0 ${-baseline} 0"/>
-    </xacro:camera_macro>
-  </xacro:macro>
-  <!-- MYNT Camera has two cameras in it; We have to handle it similarly to stereo cameras -->
-  <xacro:macro name="mynt_macro" params="namespace parent_link name update_rate hfov width height stddev baseline imu_topic imu_rate *origin">
-    <xacro:property name="camera_namespace" default="${namespace}/${name}"/>
-    <link name="${camera_namespace}/base_link">
-        <xacro:dummy_inertia />
-        <xacro:no_collision />
-    </link>
-    <joint name="${camera_namespace}/base_joint" type="fixed">
-        <xacro:insert_block name="origin" />
-        <parent link="${parent_link}" />
-        <child link="${camera_namespace}/base_link" />
-    </joint>
-    <xacro:camera_macro
-      namespace="${namespace}"
-      name="${name}/left"
-      parent_link="${camera_namespace}/base_link"
-      update_rate="${update_rate}"
-      hfov="${hfov}"
-      width="${width}"
-      height="${height}"
-      stddev="${stddev}"
-      baseline="${baseline}">
-      <origin xyz="0 0 0"/>
-    </xacro:camera_macro>
-    <!-- Right camera -->
-    <xacro:camera_macro
-      namespace="${namespace}"
-      name="${name}/right"
-      parent_link="${camera_namespace}/left_link"
-      update_rate="${update_rate}"
-      hfov="${hfov}"
-      width="${width}"
-      height="${height}"
-      stddev="${stddev}"
-      baseline="${baseline}">
-      <origin xyz="0 ${-baseline} 0"/>
-    </xacro:camera_macro>
-    <!-- IMU needs added here rather than completely separately because its link/frame need to be relative from the camera itself -->
-    <!-- TODO: I copied these numbers over from the original macro. Fill in values for the MYNT imu. -->
-    <!-- If this macro is running, we can safely assume that this value in the .yaml exists, because if this is running we have a mynt camera initially. -->
-    <xacro:imu_plugin_macro
-      namespace="${camera_namespace}"
-      imu_suffix=""
-      parent_link="${camera_namespace}/base_link"
-      imu_topic="${imu_topic}"
-      gyroscope_noise_density="0.0003394"
-      gyroscope_random_walk="0.000038785"
-      gyroscope_bias_correlation_time="1000.0"
-      gyroscope_turn_on_bias_sigma="0.0087"
-      accelerometer_noise_density="0.004"
-      accelerometer_random_walk="0.006"
-      accelerometer_bias_correlation_time="300.0"
-      accelerometer_turn_on_bias_sigma="0.1960"
-      orientation_noise="0.01"
-      enable_local_ned_frame="false"
-      reference_frame="${inertial_reference_frame}"
-      update_rate="${imu_rate}">
-      <!-- Halfway between the two cameras -->
-      <origin xyz="0 ${-baseline/2} 0" rpy="${0.5*pi} 0 ${-0.5*pi}"/>
-    </xacro:imu_plugin_macro>
-    <!-- TODO: Add gazebo camera plugin http://gazebosim.org/tutorials/?tut=ros_depth_camera -->
-    <!-- imu plugin is already here; We launch the mynt imu with the same macro as our original macro -->
-  </xacro:macro>
-  <xacro:macro name="dvl_single_sonar" params="namespace suffix index pitch yaw update_rate">
-    <link name="${namespace}/dvl${suffix}_sonar${index}_link">
-      <xacro:dummy_inertia/>
-      <xacro:no_collision/>
-    </link>
-    <joint name="${namespace}/dvl${suffix}_sonar${index}_joint" type="fixed">
-      <origin xyz="0 0 0" rpy="0 ${pitch} ${yaw}"/>
-      <parent link="${namespace}/dvl${suffix}_link" />
-      <child link="${namespace}/dvl${suffix}_sonar${index}_link" />
-    </joint>
-    <gazebo reference="${namespace}/dvl${suffix}_sonar${index}_link">
-      <sensor type="ray" name="dvl${suffix}_sonar${index}">
-        <pose>0 0 0 0 0 0</pose>
-        <update_rate>${update_rate}</update_rate>
-        <visualize>false</visualize>
-        <ray>
-          <scan>
-            <horizontal>
-              <samples>3</samples>
-              <resolution>1</resolution>
-              <min_angle>-0.03</min_angle>
-              <max_angle>0.03</max_angle>
-            </horizontal>
-            <vertical>
-              <samples>3</samples>
-              <resolution>1</resolution>
-              <min_angle>-0.03</min_angle>
-              <max_angle>0.03</max_angle>
-            </vertical>
-          </scan>
-          <range>
-            <min>0.55</min>
-            <max>10</max>
-            <resolution>0.01</resolution>
-          </range>
-        </ray>
-        <plugin filename="libgazebo_ros_range.so" name="dvl${suffix}_sonar${index}">
-          <gaussianNoise>0.005</gaussianNoise>
-          <alwaysOn>true</alwaysOn>
-          <updateRate>${update_rate}</updateRate>
-          <topicName>${topic}_sonar${index}</topicName>
-          <frameName>${namespace}/dvl${suffix}_sonar${index}_link</frameName>
-          <fov>0.06</fov>
-          <radiation>ultrasound</radiation>
-        </plugin>
-      </sensor>
-    </gazebo>
-  </xacro:macro>
-  <xacro:macro name="dvl_plugin_macro"
-    params="namespace suffix parent_link topic scale *origin update_rate
+                </plugin>
+                <always_on>1</always_on>
+                <update_rate>${update_rate}</update_rate>
+            </sensor>
+        </gazebo>
+    </xacro:macro>
+    <xacro:macro name="stereo_macro" params="namespace parent_link name update_rate hfov width height stddev baseline *origin">
+        <xacro:camera_macro namespace="${namespace}" name="${name}/left" parent_link="${parent_link}" update_rate="${update_rate}" hfov="${hfov}" width="${width}" height="${height}" stddev="${stddev}" baseline="${baseline}">
+            <xacro:insert_block name="origin" />
+        </xacro:camera_macro>
+        <xacro:camera_macro namespace="${namespace}" name="${name}/right" parent_link="${namespace}/${name}/left_link" update_rate="${update_rate}" hfov="${hfov}" width="${width}" height="${height}" stddev="${stddev}" baseline="${baseline}">
+            <origin xyz="0 ${-baseline} 0" />
+        </xacro:camera_macro>
+    </xacro:macro>
+    <!-- MYNT Camera has two cameras in it; We have to handle it similarly to stereo cameras -->
+    <xacro:macro name="mynt_macro" params="namespace parent_link name update_rate hfov width height stddev baseline imu_topic imu_rate *origin">
+        <xacro:property name="camera_namespace" default="${namespace}/${name}" />
+        <link name="${camera_namespace}/base_link">
+            <xacro:dummy_inertia />
+            <xacro:no_collision />
+        </link>
+        <joint name="${camera_namespace}/base_joint" type="fixed">
+            <xacro:insert_block name="origin" />
+            <parent link="${parent_link}" />
+            <child link="${camera_namespace}/base_link" />
+        </joint>
+        <xacro:camera_macro namespace="${namespace}" name="${name}_left" parent_link="${camera_namespace}/base_link" update_rate="${update_rate}" hfov="${hfov}" width="${width}" height="${height}" stddev="${stddev}" baseline="${baseline}">
+            <origin xyz="0 0 0" />
+        </xacro:camera_macro>
+        <!-- Right camera -->
+        <xacro:camera_macro namespace="${namespace}" name="${name}_right" parent_link="${camera_namespace}/left_link" update_rate="${update_rate}" hfov="${hfov}" width="${width}" height="${height}" stddev="${stddev}" baseline="${baseline}">
+            <origin xyz="0 ${-baseline} 0" />
+        </xacro:camera_macro>
+        <!-- IMU needs added here rather than completely separately because its link/frame need to be relative from the camera itself -->
+        <!-- TODO: I copied these numbers over from the original macro. Fill in values for the MYNT imu. -->
+        <!-- If this macro is running, we can safely assume that this value in the .yaml exists, because if this is running we have a mynt camera initially. -->
+        <xacro:imu_plugin_macro namespace="${camera_namespace}" imu_suffix="" parent_link="${camera_namespace}/base_link" imu_topic="${imu_topic}" gyroscope_noise_density="0.0003394" gyroscope_random_walk="0.000038785" gyroscope_bias_correlation_time="1000.0" gyroscope_turn_on_bias_sigma="0.0087" accelerometer_noise_density="0.004" accelerometer_random_walk="0.006" accelerometer_bias_correlation_time="300.0" accelerometer_turn_on_bias_sigma="0.1960" orientation_noise="0.01" enable_local_ned_frame="false" reference_frame="${inertial_reference_frame}" update_rate="${imu_rate}">
+            <!-- Halfway between the two cameras -->
+            <origin xyz="0 ${-baseline/2} 0" rpy="${0.5*pi} 0 ${-0.5*pi}" />
+        </xacro:imu_plugin_macro>
+        <!-- TODO: Add gazebo camera plugin http://gazebosim.org/tutorials/?tut=ros_depth_camera -->
+        <!-- imu plugin is already here; We launch the mynt imu with the same macro as our original macro -->
+    </xacro:macro>
+    <xacro:macro name="dvl_single_sonar" params="namespace suffix index pitch yaw update_rate">
+        <link name="${namespace}/dvl${suffix}_sonar${index}_link">
+            <xacro:dummy_inertia />
+            <xacro:no_collision />
+        </link>
+        <joint name="${namespace}/dvl${suffix}_sonar${index}_joint" type="fixed">
+            <origin xyz="0 0 0" rpy="0 ${pitch} ${yaw}" />
+            <parent link="${namespace}/dvl${suffix}_link" />
+            <child link="${namespace}/dvl${suffix}_sonar${index}_link" />
+        </joint>
+        <gazebo reference="${namespace}/dvl${suffix}_sonar${index}_link">
+            <sensor type="ray" name="dvl${suffix}_sonar${index}">
+                <pose>0 0 0 0 0 0</pose>
+                <update_rate>${update_rate}</update_rate>
+                <visualize>false</visualize>
+                <ray>
+                    <scan>
+                        <horizontal>
+                            <samples>3</samples>
+                            <resolution>1</resolution>
+                            <min_angle>-0.03</min_angle>
+                            <max_angle>0.03</max_angle>
+                        </horizontal>
+                        <vertical>
+                            <samples>3</samples>
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
Commit message: Added Hydrodynamics system and change groundtruth pose to be commented out

File: urdf/robot_base.xacro (robot description, xacro)
@@ -42,11 +42,34 @@
     <!-- Set up hydrodynamic plugin -->
     <gazebo>
-      <plugin name="uuv_plugin" filename="libuuv_underwater_object_ros_plugin.so">
+      <!-- TODO: ADD Buoyancy System -->
+      <plugin filename="ignition-gazebo-hydrodynamics-system" name="ignition::gazebo::systems::Hydrodynamics">
+          <link_name>base_link</link_name>
+          <xacro:property name="lin" value="${config['linear_damping']}"/>
+          <xacro:property name="quad" value="${config['quadratic_damping']}"/>
+          <xDotU>0</xDotU>
+          <yDotV>0</yDotV>
+          <zDotW>0</zDotW>
+          <kDotP>0</kDotP>
+          <mDotQ>0</mDotQ>
+          <nDotR>0</nDotR>
+          <xUU>${quad[0]}</xUU>
+          <xU>${lin[0]}</xU>
+          <yVV>${quad[1]}</yVV>
+          <yV>${lin[1]}</yV>
+          <zWW>${quad[2]}</zWW>
+          <zW>${lin[2]}</zW>
+          <kPP>${quad[3]}</kPP>
+          <kP>${lin[3]}</kP>
+          <mQQ>${quad[4]}</mQQ>
+          <mQ>${lin[4]}</mQ>
+          <nRR>${quad[5]}</nRR>
+          <nR>${lin[5]}</nR>
+      </plugin>
+      <!-- <plugin name="uuv_plugin" filename="libuuv_underwater_object_ros_plugin.so">
         <fluid_density>1000</fluid_density>
         <flow_velocity_topic>hydrodynamics/current_velocity</flow_velocity_topic>
         <debug>$(arg debug)</debug>
-        <!-- Adding the hydrodynamic and hydrostatic parameters for the vehicle-->
         <xacro:puddles_hydro_model namespace="$(arg namespace)"/>
-      </plugin>
+      </plugin> -->
     </gazebo>
     <xacro:include filename="$(find riptide_descriptions2)/urdf/robot_sensors.xacro" />

File: urdf/snippets.xacro (robot description, xacro)
@@ -28,5 +28,5 @@
             <limit effort="0" lower="0" upper="0" velocity="0" />
         </joint>
-        <gazebo>
+        <!-- <gazebo>
             <plugin name="pose_3d_plugin" filename="libuuv_gazebo_ros_pose_gt_plugin.so">
                 <ros>
@@ -42,5 +42,5 @@
                 <publish_ned_odom>false</publish_ned_odom>
             </plugin>
-        </gazebo>
+        </gazebo> -->
     </xacro:macro>
     <!-- TODO: Add camera distortion -->
