Commit message: Fixing stupid inertia issue

File: urdf/snippets.xacro (robot description, xacro)
@@ -4,6 +4,6 @@
   <xacro:macro name="dummy_inertia">
     <inertial>
-      <mass value=".001" />
-      <inertia ixx="0" ixy="0.0" ixz="0.0" iyy="0" iyz="0.0" izz="0" />
+      <mass value="0.00001" />
+      <inertia ixx="0.000001" ixy="0.0" ixz="0.0" iyy="0.000001" iyz="0.0" izz="0.000001" />
     </inertial>
   </xacro:macro>

Commit message: Tweaked mynt namespace stuff

File: urdf/snippets.xacro (robot description, xacro)
@@ -134,5 +134,5 @@
   <xacro:macro name="mynt_macro" params="namespace parent_link name update_rate hfov width height stddev baseline imu_topic imu_rate *origin">
     <!-- Parent link is {namespace]/origin -->
-    <link name="${namespace}/${name}/base_link">
+    <link name="${namespace}/${name}_link">
         <xacro:dummy_inertia />
         <xacro:no_collision />
@@ -141,11 +141,11 @@
         <xacro:insert_block name="origin" />
         <parent link="${parent_link}" />
-        <child link="${namespace}/${name}/base_link" />
+        <child link="${namespace}/${name}_link" />
     </joint>
     <!-- Left camera -->
     <xacro:mynt_camera_macro
-      namespace="${namespace}"
-      name="${name}/left"
-      parent_link="${namespace}/${name}/base_link"
+      namespace="${namespace}/${name}"
+      name="left"
+      parent_link="${namespace}/${name}_link"
       update_rate="${update_rate}"
       hfov="${hfov}"
@@ -158,7 +158,7 @@
     <!-- Right camera -->
     <xacro:mynt_camera_macro
-      namespace="${namespace}"
-      name="${name}/right"
-      parent_link="${namespace}/${name}/base_link"
+      namespace="${namespace}/${name}"
+      name="right"
+      parent_link="${namespace}/${name}_link"
       update_rate="${update_rate}"
       hfov="${hfov}"
@@ -175,5 +175,5 @@
       namespace="${namespace}/${name}"
       imu_suffix=""
-      parent_link="${namespace}/${name}/base_link"
+      parent_link="${namespace}/${name}_link"
       imu_topic="${imu_topic}"
       gyroscope_noise_density="0.0003394"

Commit message: Improving mynt representation

File: urdf/snippets.xacro (robot description, xacro)
@@ -133,19 +133,18 @@
   <!-- MYNT Camera has two cameras in it; We have to handle it similarly to stereo cameras -->
   <xacro:macro name="mynt_macro" params="namespace parent_link name update_rate hfov width height stddev baseline imu_topic imu_rate *origin">
-    <!-- Parent link is {namespace]/origin -->
-    <link name="${namespace}/${name}_link">
+    <xacro:property name="camera_namespace" default="${namespace}/${name}"/>
+    <link name="${camera_namespace}/base_link">
         <xacro:dummy_inertia />
         <xacro:no_collision />
     </link>
-    <joint name="${namespace}/${name}_joint" type="fixed">
+    <joint name="${camera_namespace}/base_joint" type="fixed">
         <xacro:insert_block name="origin" />
         <parent link="${parent_link}" />
-        <child link="${namespace}/${name}_link" />
-    </joint>
-    <!-- Left camera -->
-    <xacro:mynt_camera_macro
-      namespace="${namespace}/${name}"
-      name="left"
-      parent_link="${namespace}/${name}_link"
+        <child link="${camera_namespace}/base_link" />
+    </joint>
+    <xacro:camera_macro
+      namespace="${namespace}"
+      name="${name}/left"
+      parent_link="${camera_namespace}/base_link"
       update_rate="${update_rate}"
       hfov="${hfov}"
@@ -154,11 +153,11 @@
       stddev="${stddev}"
       baseline="${baseline}">
-      <xacro:insert_block name="origin" />
-    </xacro:mynt_camera_macro>
+      <origin xyz="0 0 0"/>
+    </xacro:camera_macro>
     <!-- Right camera -->
-    <xacro:mynt_camera_macro
-      namespace="${namespace}/${name}"
-      name="right"
-      parent_link="${namespace}/${name}_link"
+    <xacro:camera_macro
+      namespace="${namespace}"
+      name="${name}/right"
+      parent_link="${camera_namespace}/left_link"
       update_rate="${update_rate}"
       hfov="${hfov}"
@@ -168,12 +167,12 @@
       baseline="${baseline}">
       <origin xyz="0 ${-baseline} 0"/>
-    </xacro:mynt_camera_macro>
+    </xacro:camera_macro>
     <!-- IMU needs added here rather than completely separately because its link/frame need to be relative from the camera itself -->
     <!-- TODO: I copied these numbers over from the original macro. Fill in values for the MYNT imu. -->
     <!-- If this macro is running, we can safely assume that this value in the .yaml exists, because if this is running we have a mynt camera initially. -->
     <xacro:imu_plugin_macro
-      namespace="${namespace}/${name}"
+      namespace="${camera_namespace}"
       imu_suffix=""
-      parent_link="${namespace}/${name}_link"
+      parent_link="${camera_namespace}/base_link"
       imu_topic="${imu_topic}"
       gyroscope_noise_density="0.0003394"
@@ -190,27 +189,8 @@
       update_rate="${imu_rate}">
       <!-- Halfway between the two cameras -->
-      <origin xyz="0 ${-baseline/2} 0" />
+      <origin xyz="0 ${-baseline/2} 0" rpy="${0.5*pi} 0 ${-0.5*pi}"/>
     </xacro:imu_plugin_macro>
     <!-- TODO: Add gazebo camera plugin http://gazebosim.org/tutorials/?tut=ros_depth_camera -->
     <!-- imu plugin is already here; We launch the mynt imu with the same macro as our original macro -->
-  </xacro:macro>
-  <!-- TODO: Add camera distortion -->
-  <!-- This is the macro that actually defines one of the MYNT cameras -->
-  <xacro:macro name="mynt_camera_macro" params="namespace name parent_link update_rate hfov width height stddev baseline:=0 *origin">
-    <link name="${namespace}/${name}_link">
-        <xacro:dummy_inertia />
-        <xacro:no_collision />
-    </link>
-    <joint name="${namespace}/${name}_joint" type="fixed">
-        <xacro:insert_block name="origin" />
-        <parent link="${parent_link}" />
-        <child link="${namespace}/${name}_link" />
-    </joint>
-    <link name="${namespace}/${name}_optical" />
-    <joint name="${namespace}/${name}_optical_joint" type="fixed">
-      <parent link="${namespace}/${name}_link" />
-      <child link="${namespace}/${name}_optical" />
-      <origin rpy="${-pi/2} 0 ${-pi/2}"></origin>
-    </joint>
   </xacro:macro>
   <xacro:macro name="dvl_single_sonar" params="namespace suffix index pitch yaw update_rate">

Commit message: Getting rid of tf warnings

File: urdf/snippets.xacro (robot description, xacro)
@@ -341,9 +341,17 @@
       <xacro:dummy_inertia/>
     </link>
+    <link name="${namespace}/imu${imu_suffix}_revolute_link">
+      <xacro:dummy_inertia/>
+    </link>
     <!-- IMU joint -->
-    <joint name="${namespace}/imu${imu_suffix}_joint" type="revolute">
+    <joint name="${namespace}/imu${imu_suffix}_joint" type="fixed">
       <xacro:insert_block name="origin" />
       <parent link="${parent_link}" />
       <child link="${namespace}/imu${imu_suffix}_link" />
+    </joint>
+    <joint name="${namespace}/imu${imu_suffix}_revolute_joint" type="revolute">
+      <xacro:insert_block name="origin" />
+      <parent link="${parent_link}" />
+      <child link="${namespace}/imu${imu_suffix}_revolute_link" />
       <limit upper="0" lower="0" effort="0" velocity="0" />
       <axis xyz="1 0 0"/>
@@ -354,6 +362,6 @@
            https://github.com/ethz-asl/kalibr/wiki/IMU-Noise-Model-and-Intrinsics -->
         <robot_namespace>${namespace}</robot_namespace> <!-- (string, required): ros namespace in which the messages are published -->
-        <link_name>${namespace}/imu${imu_suffix}_link</link_name> <!-- (string, required): name of the body which holds the IMU sensor -->
-        <sensor_topic>${imu_topic}</sensor_topic> <!-- (string): name of the sensor output topic and prefix of service names (defaults to imu) -->
+        <link_name>${namespace}/imu${imu_suffix}_revolute_link</link_name> <!-- (string, required): name of the body which holds the IMU sensor -->
+        <sensor_topic>${imu_topic}/sim</sensor_topic> <!-- (string): name of the sensor output topic and prefix of service names (defaults to imu) -->
         <gyroscope_noise_density>${gyroscope_noise_density}</gyroscope_noise_density> <!-- Gyroscope noise density (two-sided spectrum) [rad/s/sqrt(Hz)] -->
         <gyroscope_random_walk>${gyroscope_random_walk}</gyroscope_random_walk> <!-- Gyroscope bias random walk [rad/s/s/sqrt(Hz)] -->

Commit message: calculated thrust coeficient, may be too high

File: urdf/snippets.xacro (robot description, xacro)
@@ -333,21 +333,17 @@
             <xacro:no_collision />
         </link>
-        <gazebo>
-            <plugin name="${namespace}_${thruster_id}_thruster_model" filename="libuuv_thruster_ros_plugin.so">
-                <linkName>${namespace}/thruster_${thruster_id}</linkName>
-                <jointName>${namespace}/thruster_${thruster_id}_joint</jointName>
-                <thrusterID>${thruster_id}</thrusterID>
-                <dynamics>
-                    <type>ZeroOrder</type>
-                </dynamics>
-                <conversion>
-                    <type>Basic</type>
-                    <rotorConstant>${rotor_constant}</rotorConstant>
-                </conversion>
-            </plugin>
-        </gazebo>
-        <gazebo reference="${namespace}/thruster_${thruster_id}">
-            <selfCollide>false</selfCollide>
-        </gazebo>
+        <plugin
+            filename="ignition-gazebo-thruster-system"
+            name="ignition::gazebo::systems::Thruster">
+            <namespace>${namespace}</namespace>
+            <joint_name>${namespace}/thruster_${thruster_id}_joint</joint_name>
+            <!-- used the docs from blue robotics to generate this
+            Calculated from this equation in desmos \frac{3.96\cdot9.81}{1000\cdot3088^{2}\cdot0.007628^{4}}
+            3.96 is force in N, 3088 is prop rpm, blade diameter is 0.007628 m, and fluid density is 1000 kg/m^3 -->
+            <thrust_coefficient>1.20328</thrust_coefficient>
+            <fluid_density>1000</fluid_density>
+            <!-- prop diameter is 72.28 mm -->
+            <propeller_diameter>0.007628</propeller_diameter>
+        </plugin>
     </xacro:macro>
     <xacro:macro name="default_joint_state_publisher" params="namespace update_rate">

Commit message: updated dvl single sonar macro

File: urdf/snippets.xacro (robot description, xacro)
@@ -15,4 +15,49 @@
             <origin xyz="0 0 0" rpy="0 ${0.5*pi} 0" />
         </collision>
+    </xacro:macro>
+    <xacro:macro name="dvl_single_sonar" params="namespace suffix index pitch yaw update_rate">
+        <link name="${namespace}/dvl${suffix}_sonar${index}_link">
+            <xacro:dummy_inertia />
+            <xacro:no_collision />
+        </link>
+        <joint name="${namespace}/dvl${suffix}_sonar${index}_joint" type="fixed">
+            <origin xyz="0 0 0" rpy="0 ${pitch} ${yaw}" />
+            <parent link="${namespace}/dvl${suffix}_link" />
+            <child link="${namespace}/dvl${suffix}_sonar${index}_link" />
+        </joint>
+        <frame name="${namespace}/dvl${suffix}_sonar${index}_link">
+            <!-- <pose>0.8 0 0.5 0 0 0</pose> -->
+        </frame>
+        <plugin
+            filename="libignition-gazebo-sensors-system.so"
+            name="ignition::gazebo::systems::Sensors">
+            <render_engine>ogre2</render_engine>
+        </plugin>
+        <sensor name="dvl${suffix}_sonar${index}" type='gpu_lidar'>
+            <pose relative_to="${namespace}/dvl${suffix}_sonar${index}_link">0 0 0 0 0 0</pose>
+            <update_rate>${update_rate}</update_rate>
+            <ray>
+                <scan>
+                    <horizontal>
+                        <samples>3</samples>
+                        <resolution>1</resolution>
+                        <min_angle>-0.03</min_angle>
+                        <max_angle>0.03</max_angle>
+                    </horizontal>
+                    <vertical>
+                        <samples>3</samples>
+                        <resolution>1</resolution>
+                        <min_angle>-0.03</min_angle>
+                        <max_angle>0.03</max_angle>
+                    </vertical>
+                </scan>
+                <range>
+                    <min>0.55</min>
+                    <max>10</max>
+                    <resolution>0.01</resolution>
+                </range>
+            </ray>
+            <visualize>false</visualize>
+        </sensor>
     </xacro:macro>
     <!-- Ground truth position -->
