Commit message: purge all of the unused simulation constants

File: urdf/robot.gazebo.xacro (robot description, xacro)
@@ -1,30 +1,7 @@
 <?xml version="1.0"?>
 <robot xmlns:xacro="http://www.ros.org/wiki/xacro">
-    <xacro:property name="lin" value="${config['linear_damping']}"/>
-    <xacro:property name="quad" value="${config['quadratic_damping']}"/>
     <!-- All hydro parameters for any links that have them -->
     <xacro:macro name="puddles_hydro_model" params="namespace">
         <link name="${namespace}/base_link">
-            <volume>${config['volume']}</volume>
-            <!-- COB is relative to center of base_link, thus the math -->
-            <center_of_buoyancy>${config['cob'][0]-config['com'][0]} ${config['cob'][1]-config['com'][1]} ${config['cob'][2]-config['com'][2]}</center_of_buoyancy>
-            <hydrodynamic_model>
-                <!--clairedune.kippou.fr/Fossen.pdf-->
-                <type>fossen</type>
-                <added_mass>
-                    0 0 0 0 0 0
-                    0 0 0 0 0 0
-                    0 0 0 0 0 0
-                    0 0 0 0 0 0
-                    0 0 0 0 0 0
-                    0 0 0 0 0 0
-                </added_mass>
-                <linear_damping>
-                    ${lin[0]} ${lin[1]} ${lin[2]} ${lin[3]} ${lin[4]} ${lin[5]}
-                </linear_damping>
-                <quadratic_damping>
-                    ${quad[0]} ${quad[1]} ${quad[2]} ${quad[3]} ${quad[4]} ${quad[5]}
-                </quadratic_damping>
-            </hydrodynamic_model>
         </link>
     </xacro:macro>

File: urdf/robot_actuators.xacro (robot description, xacro)
@@ -20,6 +20,5 @@
         namespace="${namespace}"
         thruster_id="${index}"
-        mesh_filename="${prop_file}"
-        rotor_constant="${config['rotor_constant']}">
+        mesh_filename="${prop_file}">
         <origin xyz="${thruster['pose'][0]} ${thruster['pose'][1]} ${thruster['pose'][2]}"
                 rpy="${thruster['pose'][3]} ${thruster['pose'][4]} ${thruster['pose'][5]}"/>

File: urdf/robot_base.xacro (robot description, xacro)
@@ -40,37 +40,4 @@
       <origin xyz="${config['com'][0]} ${config['com'][1]} ${config['com'][2]}" rpy="0 0 0"/>
     </joint>
-    <!-- Set up hydrodynamic plugin -->
-    <gazebo>
-      <!-- TODO: ADD Buoyancy System -->
-      <plugin filename="ignition-gazebo-hydrodynamics-system" name="ignition::gazebo::systems::Hydrodynamics">
-          <link_name>${namespace}/base_link</link_name>
-          <xacro:property name="lin" value="${config['linear_damping']}"/>
-          <xacro:property name="quad" value="${config['quadratic_damping']}"/>
-          <xDotU>0</xDotU>
-          <yDotV>0</yDotV>
-          <zDotW>0</zDotW>
-          <kDotP>0</kDotP>
-          <mDotQ>0</mDotQ>
-          <nDotR>0</nDotR>
-          <xUU>${quad[0]}</xUU>
-          <xU>${lin[0]}</xU>
-          <yVV>${quad[1]}</yVV>
-          <yV>${lin[1]}</yV>
-          <zWW>${quad[2]}</zWW>
-          <zW>${lin[2]}</zW>
-          <kPP>${quad[3]}</kPP>
-          <kP>${lin[3]}</kP>
-          <mQQ>${quad[4]}</mQQ>
-          <mQ>${lin[4]}</mQ>
-          <nRR>${quad[5]}</nRR>
-          <nR>${lin[5]}</nR>
-      </plugin>
-      <!-- <plugin name="uuv_plugin" filename="libuuv_underwater_object_ros_plugin.so">
-        <fluid_density>1000</fluid_density>
-        <flow_velocity_topic>hydrodynamics/current_velocity</flow_velocity_topic>
-        <debug>$(arg debug)</debug>
-        <xacro:puddles_hydro_model namespace="$(arg namespace)"/>
-      </plugin> -->
-    </gazebo>
     <xacro:include filename="$(find riptide_descriptions2)/urdf/robot_sensors.xacro" />
     <xacro:include filename="$(find riptide_descriptions2)/urdf/robot_actuators.xacro" />

File: urdf/robot_sensors.xacro (robot description, xacro)
@@ -3,8 +3,4 @@
   <!-- Everything here is ENU frame -->
   <xacro:property name="dvl" value="${config['dvl']}"/>
-  <xacro:default_joint_state_publisher
-  namespace="${namespace}"
-  update_rate="${dvl['rate']}" >
-  </xacro:default_joint_state_publisher>
   <!-- DVL  -->
   <!-- TODO: restore below if when xacro releases 1.14.4 -->
@@ -14,11 +10,5 @@
       namespace="${namespace}"
       suffix=""
-      parent_link="${namespace}/origin"
-      topic="${dvl['topic']}"
-      scale="1"
-      update_rate="${dvl['rate']}"
-      reference_frame="${inertial_reference_frame}"
-      noise_sigma="${dvl['sigma']}"
-      noise_amplitude="1">
+      parent_link="${namespace}/origin">
       <origin xyz="${dvl['pose'][0]} ${dvl['pose'][1]} ${dvl['pose'][2]}"
               rpy="${dvl['pose'][3]} ${dvl['pose'][4]} ${dvl['pose'][5]}"/>
@@ -32,13 +22,5 @@
       namespace="${namespace}"
       suffix=""
-      parent_link="${namespace}/origin"
-      topic="${depth['topic']}"
-      update_rate="${depth['rate']}"
-      range="300"
-      noise_sigma="${depth['sigma'] * 9.80638}"
-      noise_amplitude="1"
-      estimateDepth="false"
-      standardPressure="101.325"
-      kPaPerM="9.80638">
+      parent_link="${namespace}/origin">
       <origin xyz="${depth['pose'][0]} ${depth['pose'][1]} ${depth['pose'][2]}"
               rpy="${depth['pose'][3]} ${depth['pose'][4]} ${depth['pose'][5]}"/>
@@ -53,18 +35,5 @@
       namespace="${namespace}"
       imu_suffix=""
-      parent_link="${namespace}/origin"
-      imu_topic="${namespace}/${imu['topic']}"
-      gyroscope_noise_density="0.0003394"
-      gyroscope_random_walk="0.000038785"
-      gyroscope_bias_correlation_time="1000.0"
-      gyroscope_turn_on_bias_sigma="0.0087"
-      accelerometer_noise_density="0.004"
-      accelerometer_random_walk="0.006"
-      accelerometer_bias_correlation_time="300.0"
-      accelerometer_turn_on_bias_sigma="0.1960"
-      orientation_noise="0.01"
-      enable_local_ned_frame="false"
-      reference_frame="${inertial_reference_frame}"
-      update_rate="${imu['rate']}">
+      parent_link="${namespace}/origin">
       <origin xyz="${imu['pose'][0]} ${imu['pose'][1]} ${imu['pose'][2]}"
               rpy="${imu['pose'][3]} ${imu['pose'][4]} ${imu['pose'][5]}"/>
@@ -85,11 +54,5 @@
           namespace="${namespace}"
           parent_link="${namespace}/origin"
-          name="${camera['name']}"
-          update_rate="${camera['rate']}"
-          hfov="${camera['hfov']}"
-          width="${camera['width']}"
-          height="${camera['height']}"
-          stddev="${camera['stddev']}"
-          baseline="${camera['baseline']}">
+          name="${camera['name']}">
           <origin xyz="${camera['pose'][0]} ${camera['pose'][1]} ${camera['pose'][2]}"
                   rpy="${camera['pose'][3]} ${camera['pose'][4]} ${camera['pose'][5]}"/>
@@ -102,10 +65,5 @@
             namespace="${namespace}"
             name="${camera['name']}"
-            parent_link="${namespace}/origin"
-            update_rate="${camera['rate']}"
-            hfov="${camera['hfov']}"
-            width="${camera['width']}"
-            height="${camera['height']}"
-            stddev="${camera['stddev']}">
+            parent_link="${namespace}/origin">
             <origin xyz="${camera['pose'][0]} ${camera['pose'][1]} ${camera['pose'][2]}"
                     rpy="${camera['pose'][3]} ${camera['pose'][4]} ${camera['pose'][5]}"/>
@@ -115,23 +73,4 @@
         <!-- Suffix isn't set here because right now we just have one, but you should just need to change the suffix for each and it'll work. -->
         <xacro:unless value="${camera['type'] == 'mono'}">
-          <!-- <xacro:include filename="$(find zed_wrapper)/urdf/zed_macro.urdf.xacro" /> -->
-          <!-- <xacro:zed_camera name="${camera['name']}" model="${camera['model']}" parent="${namespace}/base_link" >
-            <origin xyz="${camera['pose'][0]} ${camera['pose'][1]} ${camera['pose'][2]}" rpy="${camera['pose'][3]} ${camera['pose'][4]} ${camera['pose'][5]}" />
-          </xacro:zed_camera> -->
-          <!-- <xacro:mynt_macro
-            namespace="${namespace}"
-            name="${camera['name']}"
-            parent_link="${namespace}/origin"
-            update_rate="${camera['rate']}"
-            hfov="${camera['hfov']}"
-            width="${camera['width']}"
-            height="${camera['height']}"
-            stddev="${camera['stddev']}"
-            baseline="${camera['baseline']}"
-            imu_topic="${camera['imu_topic']}"
-            imu_rate="${camera['imu_rate']}">
-            <origin xyz="${camera['pose'][0]} ${camera['pose'][1]} ${camera['pose'][2]}"
-                    rpy="${camera['pose'][3]} ${camera['pose'][4]} ${camera['pose'][5]}"/>
-          </xacro:mynt_macro> -->
         </xacro:unless>
       </xacro:unless>
