Commit message: purge all of the unused simulation constants

File: urdf/snippets.xacro (robot description, xacro)
@@ -16,49 +16,4 @@
         </collision>
     </xacro:macro>
-    <xacro:macro name="dvl_single_sonar" params="namespace suffix index pitch yaw update_rate">
-        <link name="${namespace}/dvl${suffix}_sonar${index}_link">
-            <xacro:dummy_inertia />
-            <xacro:no_collision />
-        </link>
-        <joint name="${namespace}/dvl${suffix}_sonar${index}_joint" type="fixed">
-            <origin xyz="0 0 0" rpy="0 ${pitch} ${yaw}" />
-            <parent link="${namespace}/dvl${suffix}_link" />
-            <child link="${namespace}/dvl${suffix}_sonar${index}_link" />
-        </joint>
-        <frame name="${namespace}/dvl${suffix}_sonar${index}_link">
-            <!-- <pose>0.8 0 0.5 0 0 0</pose> -->
-        </frame>
-        <plugin
-            filename="libignition-gazebo-sensors-system.so"
-            name="ignition::gazebo::systems::Sensors">
-            <render_engine>ogre2</render_engine>
-        </plugin>
-        <sensor name="dvl${suffix}_sonar${index}" type='gpu_lidar'>
-            <pose relative_to="${namespace}/dvl${suffix}_sonar${index}_link">0 0 0 0 0 0</pose>
-            <update_rate>${update_rate}</update_rate>
-            <ray>
-                <scan>
-                    <horizontal>
-                        <samples>3</samples>
-                        <resolution>1</resolution>
-                        <min_angle>-0.03</min_angle>
-                        <max_angle>0.03</max_angle>
-                    </horizontal>
-                    <vertical>
-                        <samples>3</samples>
-                        <resolution>1</resolution>
-                        <min_angle>-0.03</min_angle>
-                        <max_angle>0.03</max_angle>
-                    </vertical>
-                </scan>
-                <range>
-                    <min>0.55</min>
-                    <max>10</max>
-                    <resolution>0.01</resolution>
-                </range>
-            </ray>
-            <visualize>false</visualize>
-        </sensor>
-    </xacro:macro>
     <!-- Ground truth position -->
     <xacro:macro name="default_pose_3d_macro" params="namespace parent_link inertial_reference_frame">
@@ -73,22 +28,6 @@
             <limit effort="0" lower="0" upper="0" velocity="0" />
         </joint>
-        <!-- <gazebo>
-            <plugin name="pose_3d_plugin" filename="libuuv_gazebo_ros_pose_gt_plugin.so">
-                <ros>
-                    <namespace>${namespace}</namespace>
-                </ros>
-                <link_name>${namespace}/base_link</link_name>
-                <sensor_topic>pose_gt</sensor_topic>
-                <static_reference_frame>${inertial_reference_frame}</static_reference_frame>
-                <noise_sigma>0</noise_sigma>
-                <noise_amplitude>0</noise_amplitude>
-                <update_rate>20</update_rate>
-                <enable_gazebo_messages>false</enable_gazebo_messages>
-                <publish_ned_odom>false</publish_ned_odom>
-            </plugin>
-        </gazebo> -->
     </xacro:macro>
-    <!-- TODO: Add camera distortion -->
-    <xacro:macro name="camera_macro" params="namespace name parent_link update_rate hfov width height stddev baseline:=0 *origin">
+    <xacro:macro name="camera_macro" params="namespace name parent_link *origin">
         <link name="${namespace}/${name}_link">
             <xacro:dummy_inertia />
@@ -106,154 +45,6 @@
             <origin rpy="${-pi/2} 0 ${-pi/2}"></origin>
         </joint>
-        <!-- <ignition reference="${namespace}/${name}_link"> -->
-            <sensor name="${name}" type="camera">
-                <camera>
-                    <topic>${namespace}/${name}</topic>
-                    <horizontal_fov>${hfov}</horizontal_fov>
-                    <image>
-                        <width>${width}</width>
-                        <height>${height}</height>
-                        <format>R8G8B8</format>
-                    </image>
-                    <clip>
-                        <near>0.05</near>
-                        <far>3000</far>
-                    </clip>
-                    <noise>
-                        <type>gaussian</type>
-                        <mean>0.0</mean>
-                        <stddev>${stddev}</stddev>
-                    </noise>
-                </camera>
-                <!-- <plugin name="${name}_controller" filename="libgazebo_ros_camera.so">
-                    <alwaysOn>true</alwaysOn>
-                    <ros>
-                        <camera_name>${name}</camera_name>
-                        <remapping>${name}/image_raw:=${namespace}/${name}/image_raw</remapping>
-                        <remapping>${name}/image_raw/compressed:=${namespace}/${name}/image_raw/compressed</remapping>
-                        <remapping>${name}/camera_info:=${namespace}/${name}/camera_info</remapping>
-                    </ros>
-                    <frameName>${namespace}/${name}_optical</frameName>
-                    <hackBaseline>${baseline}</hackBaseline>
-                </plugin> -->
-                <always_on>1</always_on>
-                <update_rate>${update_rate}</update_rate>
-            </sensor>
-        <!-- </ignition> -->
     </xacro:macro>
-    <xacro:macro name="stereo_macro" params="namespace parent_link name update_rate hfov width height stddev baseline *origin">
-        <xacro:camera_macro namespace="${namespace}/${name}" name="left" parent_link="${parent_link}" update_rate="${update_rate}" hfov="${hfov}" width="${width}" height="${height}" stddev="${stddev}" baseline="${baseline}">
-            <xacro:insert_block name="origin" />
-        </xacro:camera_macro>
-        <xacro:camera_macro namespace="${namespace}" name="right" parent_link="${namespace}/${name}/left_link" update_rate="${update_rate}" hfov="${hfov}" width="${width}" height="${height}" stddev="${stddev}" baseline="${baseline}">
-            <origin xyz="0 ${-baseline} 0" />
-        </xacro:camera_macro>
-    </xacro:macro>
-    <!-- MYNT Camera has two cameras in it; We have to handle it similarly to stereo cameras -->
-    <xacro:macro name="mynt_macro" params="namespace parent_link name update_rate hfov width height stddev baseline imu_topic imu_rate *origin">
-        <xacro:property name="camera_namespace" default="${namespace}/${name}" />
-        <link name="${camera_namespace}/base_link">
-            <xacro:dummy_inertia />
-            <xacro:no_collision />
-        </link>
-        <joint name="${camera_namespace}/base_joint" type="fixed">
-            <xacro:insert_block name="origin" />
-            <parent link="${parent_link}" />
-            <child link="${camera_namespace}/base_link" />
-        </joint>
-        <xacro:camera_macro namespace="${namespace}/${name}" name="left" parent_link="${camera_namespace}/base_link" update_rate="${update_rate}" hfov="${hfov}" width="${width}" height="${height}" stddev="${stddev}" baseline="${baseline}">
-            <origin xyz="0 0 0" />
-            <!-- <ignition reference="${namespace}/${name}_link"> -->
-                <!-- <sensor name="${name}" type="depth_camera">
-                    <topic>${namespace}/${name}</topic>
-                    <camera>
-                      <horizontal_fov>${hfov}</horizontal_fov>
-                      <image>
-                        <width>${width}</width>
-                        <height>${height}</height>
-                        <format>R_FLOAT32</format>
-                      </image>
-                      <clip>
-                        <near>0.05</near>
-                        <far>3000</far>
-                      </clip>
-                      <noise>
-                        <type>gaussian</type>
-                        <mean>0.0</mean>
-                        <stddev>${stddev}</stddev>
-                    </noise>
-                    </camera>
-                    <update_rate>${update_rate}</update_rate>
-                </sensor> -->
-            <!-- </ignition> -->
-        </xacro:camera_macro>
-        <!-- Right camera -->
-        <xacro:camera_macro namespace="${namespace}/${name}" name="right" parent_link="${camera_namespace}/left_link" update_rate="${update_rate}" hfov="${hfov}" width="${width}" height="${height}" stddev="${stddev}" baseline="${baseline}">
-            <origin xyz="0 ${-baseline} 0" />
-        </xacro:camera_macro>
-        <!-- IMU needs added here rather than completely separately because its link/frame need to be relative from the camera itself -->
-        <!-- TODO: I copied these numbers over from the original macro. Fill in values for the MYNT imu. -->
-        <!-- If this macro is running, we can safely assume that this value in the .yaml exists, because if this is running we have a mynt camera initially. -->
-        <xacro:imu_plugin_macro namespace="${camera_namespace}" imu_suffix="" parent_link="${camera_namespace}/base_link" imu_topic="${imu_topic}" gyroscope_noise_density="0.0003394" gyroscope_random_walk="0.000038785" gyroscope_bias_correlation_time="1000.0" gyroscope_turn_on_bias_sigma="0.0087" accelerometer_noise_density="0.004" accelerometer_random_walk="0.006" accelerometer_bias_correlation_time="300.0" accelerometer_turn_on_bias_sigma="0.1960" orientation_noise="0.01" enable_local_ned_frame="false" reference_frame="${inertial_reference_frame}" update_rate="${imu_rate}">
-            <!-- Halfway between the two cameras -->
-            <origin xyz="0 ${-baseline/2} 0" rpy="${0.5*pi} 0 ${-0.5*pi}" />
-        </xacro:imu_plugin_macro>
-        <!-- TODO: Add gazebo camera plugin http://gazebosim.org/tutorials/?tut=ros_depth_camera -->
-        <!-- imu plugin is already here; We launch the mynt imu with the same macro as our original macro -->
-    </xacro:macro>
-    <xacro:macro name="dvl_single_sonar" params="namespace suffix index pitch yaw update_rate">
-        <link name="${namespace}/dvl${suffix}_sonar${index}_link">
-            <xacro:dummy_inertia />
-            <xacro:no_collision />
-        </link>
-        <joint name="${namespace}/dvl${suffix}_sonar${index}_joint" type="fixed">
-            <origin xyz="0 0 0" rpy="0 ${pitch} ${yaw}" />
-            <parent link="${namespace}/dvl${suffix}_link" />
-            <child link="${namespace}/dvl${suffix}_sonar${index}_link" />
-        </joint>
-        <gazebo reference="${namespace}/dvl${suffix}_sonar${index}_link">
-            <sensor type="ray" name="dvl${suffix}_sonar${index}">
-                <pose>0 0 0 0 0 0</pose>
-                <update_rate>${update_rate}</update_rate>
-                <visualize>false</visualize>
-                <ray>
-                    <scan>
-                        <horizontal>
-                            <samples>3</samples>
-                            <resolution>1</resolution>
-                            <min_angle>-0.03</min_angle>
-                            <max_angle>0.03</max_angle>
-                        </horizontal>
-                        <vertical>
-                            <samples>3</samples>
-                            <resolution>1</resolution>
-                            <min_angle>-0.03</min_angle>
-                            <max_angle>0.03</max_angle>
-                        </vertical>
-                    </scan>
-                    <range>
-                        <min>0.55</min>
-                        <max>10</max>
-                        <resolution>0.01</resolution>
-                    </range>
-                </ray>
-                <!-- <plugin filename="libgazebo_ros_ray_sensor.so" name="dvl${suffix}_sonar${index}"> TODO: COMMENTED PLUGIN
-                    <ros>
-                        <namespace>${namespace}</namespace>
-                    </ros>
-                    <gaussianNoise>0.005</gaussianNoise>
-                    <alwaysOn>true</alwaysOn>
-                    <updateRate>${update_rate}</updateRate>
-                    <topicName>${topic}_sonar${index}</topicName>
-                    <frameName>${namespace}/dvl${suffix}_sonar${index}_link</frameName>
-                    <fov>0.06</fov>
-                    <radiation_type>ultrasound</radiation_type>
-                    <output_type>sensor_msgs/Range</output_type>
-                </plugin> -->
-            </sensor>
-        </gazebo>
-    </xacro:macro>
-    <xacro:macro name="dvl_plugin_macro" params="namespace suffix parent_link topic scale *origin update_rate
-    reference_frame noise_sigma noise_amplitude">
+    <xacro:macro name="dvl_plugin_macro" params="namespace suffix parent_link *origin">
         <link name="${namespace}/dvl${suffix}_link">
             <xacro:dummy_inertia />
@@ -267,37 +58,6 @@
             <axis xyz="1 0 0" />
         </joint>
-        <xacro:dvl_single_sonar namespace="${namespace}" suffix="${suffix}" index="0" pitch="1.309" yaw="-0.7854" update_rate="${update_rate}"></xacro:dvl_single_sonar>
-        <xacro:dvl_single_sonar namespace="${namespace}" suffix="${suffix}" index="1" pitch="1.309" yaw="-2.35619" update_rate="${update_rate}"></xacro:dvl_single_sonar>
-        <xacro:dvl_single_sonar namespace="${namespace}" suffix="${suffix}" index="2" pitch="1.309" yaw="2.35619" update_rate="${update_rate}"></xacro:dvl_single_sonar>
-        <xacro:dvl_single_sonar namespace="${namespace}" suffix="${suffix}" index="3" pitch="1.309" yaw="0.7854" update_rate="${update_rate}"></xacro:dvl_single_sonar>
-        <!-- <gazebo> TODO: COMMENTED PLUGIN
-            <plugin filename="libuuv_gazebo_ros_dvl_plugin.so" name="libuuv_gazebo_dvl${suffix}_plugin">
-                <ros>
-                    <namespace>${namespace}</namespace>
-                </ros> (string, required): ros namespace in which the messages are published
-                <link_name>${namespace}/dvl${suffix}_link</link_name>
-                <sensor_topic>${topic}</sensor_topic> (string): name of the sensor output topic and prefix of service names
-                <update_rate>${update_rate}</update_rate> Update period [s]
-                <noise_sigma>${noise_sigma}</noise_sigma> std dev of velocity estimates in x, y, z [m/s]
-                <noise_amplitude>${noise_amplitude}</noise_amplitude>
-                <enable_gazebo_messages>false</enable_gazebo_messages>
-                <enable_local_ned_frame>false</enable_local_ned_frame>
-                <static_reference_frame>${reference_frame}</static_reference_frame>
-                Declaring the beams
-                <beam_link_name_0>${namespace}/dvl${suffix}_sonar0_link</beam_link_name_0>
-                <beam_link_name_1>${namespace}/dvl${suffix}_sonar1_link</beam_link_name_1>
-                <beam_link_name_2>${namespace}/dvl${suffix}_sonar2_link</beam_link_name_2>
-                <beam_link_name_3>${namespace}/dvl${suffix}_sonar3_link</beam_link_name_3>
-                Declaring the beam output topics
-                <beam_topic_0>${topic}_sonar0</beam_topic_0>
-                <beam_topic_1>${topic}_sonar1</beam_topic_1>
-                <beam_topic_2>${topic}_sonar2</beam_topic_2>
-                <beam_topic_3>${topic}_sonar3</beam_topic_3>
-            </plugin>
-        </gazebo> -->
     </xacro:macro>
-    <xacro:macro name="pressure_plugin_macro" params="namespace suffix parent_link topic update_rate
-      range noise_sigma noise_amplitude estimateDepth standardPressure kPaPerM
-      *origin">
+    <xacro:macro name="pressure_plugin_macro" params="namespace suffix parent_link *origin">
         <link name="${namespace}/pressure${suffix}_link">
             <xacro:dummy_inertia />
@@ -311,29 +71,6 @@
             <axis xyz="1 0 0" />
         </joint>
-        <!-- <gazebo> TODO: COMMENTED PLUGIN
-            <plugin filename="libuuv_gazebo_ros_subsea_pressure_plugin.so" name="libuuv_gazebo_subseapressure${suffix}_plugin">
-                <robot_namespace>${namespace}</robot_namespace> (string, required): ros namespace in which the messages are published
-                <link_name>${namespace}/pressure${suffix}_link</link_name>
-                <sensor_topic>${topic}</sensor_topic>
-                <update_rate>${update_rate}</update_rate>
-                <saturation>${range}</saturation> measurement range [kPa]
-                <noise_sigma>${noise_sigma}</noise_sigma> measurement stddev [kPa]
-                <noise_amplitude>${noise_amplitude}</noise_amplitude>
-                <estimate_depth_on>${estimateDepth}</estimate_depth_on> infer depth?
-                <standard_pressure>${standardPressure}</standard_pressure> pressure at sea level (depth 0 m) [kPa]
-                <kPa_per_meter>${kPaPerM}</kPa_per_meter> increase in pressure [kPa] per [m] in increased depth
-                <enable_gazebo_messages>false</enable_gazebo_messages>
-            </plugin>
-        </gazebo> -->
     </xacro:macro>
-    <xacro:macro name="imu_plugin_macro" params="namespace imu_suffix parent_link imu_topic
-      gyroscope_noise_density gyroscope_random_walk
-      gyroscope_bias_correlation_time gyroscope_turn_on_bias_sigma
-      accelerometer_noise_density accelerometer_random_walk
-      accelerometer_bias_correlation_time accelerometer_turn_on_bias_sigma
-      orientation_noise
-      update_rate reference_frame
-      enable_local_ned_frame
-      *origin">
+    <xacro:macro name="imu_plugin_macro" params="namespace imu_suffix parent_link *origin">
         <!-- IMU link -->
         <link name="${namespace}/imu${imu_suffix}_link">
@@ -360,6 +97,5 @@
             thruster_id
             *origin
-            mesh_filename
-            rotor_constant">
+            mesh_filename">
         <joint name="${namespace}/thruster_${thruster_id}_joint" type="continuous">
             <xacro:insert_block name="origin" />
@@ -377,28 +113,4 @@
             <xacro:no_collision />
         </link>
-        <plugin
-            filename="ignition-gazebo-thruster-system"
-            name="ignition::gazebo::systems::Thruster">
-            <namespace>${namespace}</namespace>
-            <joint_name>${namespace}/thruster_${thruster_id}_joint</joint_name>
-            <!-- used the docs from blue robotics to generate this
-            Calculated from this equation in desmos \frac{3.96\cdot9.81}{1000\cdot3088^{2}\cdot0.007628^{4}}
-            3.96 is force in N, 3088 is prop rpm, blade diameter is 0.007628 m, and fluid density is 1000 kg/m^3 -->
-            <thrust_coefficient>1.20328</thrust_coefficient>
-            <fluid_density>1000</fluid_density>
-            <!-- prop diameter is 72.28 mm -->
-            <propeller_diameter>0.007628</propeller_diameter>
-        </plugin>
-    </xacro:macro>
-    <xacro:macro name="default_joint_state_publisher" params="namespace update_rate">
-        <!-- <gazebo>
-            <plugin name="uuv_joint_state_publisher" filename="libuuv_joint_state_publisher.so">
-                <ros>
-                    <namespace>${namespace}</namespace>
-                </ros>
-                <robotNamespace>${namespace}</robotNamespace>
-                <updateRate>${update_rate}</updateRate>
-            </plugin>
-        </gazebo> -->
     </xacro:macro>
 </robot>
