Commit message: Implemented mynt macro launch conditions

File: urdf/robot_sensors.xacro (robot description, xacro)
@@ -72,4 +72,5 @@
     <xacro:if value="${cameras != []}">
       <xacro:property name="camera" value="${cameras[0]}"/>
+      <!-- Stereo Camera(s) -->
       <xacro:if value="${camera['type'] == 'stereo'}">
         <xacro:stereo_macro
@@ -87,17 +88,36 @@
         </xacro:stereo_macro>
       </xacro:if>
+      <!-- Downward Camera -->
       <xacro:unless value="${camera['type'] == 'stereo'}">
-        <xacro:camera_macro
-          namespace="${namespace}"
-          name="${camera['name']}"
-          parent_link="${namespace}/origin"
-          update_rate="${camera['rate']}"
-          hfov="${camera['hfov']}"
-          width="${camera['width']}"
-          height="${camera['height']}"
-          stddev="${camera['stddev']}">
-          <origin xyz="${camera['pose'][0]} ${camera['pose'][1]} ${camera['pose'][2]}"
-                  rpy="${camera['pose'][3]} ${camera['pose'][4]} ${camera['pose'][5]}"/>
-        </xacro:camera_macro>
+        <xacro:if value="${camera['type'] == 'downward'}">
+          <xacro:camera_macro
+            namespace="${namespace}"
+            name="${camera['name']}"
+            parent_link="${namespace}/origin"
+            update_rate="${camera['rate']}"
+            hfov="${camera['hfov']}"
+            width="${camera['width']}"
+            height="${camera['height']}"
+            stddev="${camera['stddev']}">
+            <origin xyz="${camera['pose'][0]} ${camera['pose'][1]} ${camera['pose'][2]}"
+                    rpy="${camera['pose'][3]} ${camera['pose'][4]} ${camera['pose'][5]}"/>
+          </xacro:camera_macro>
+        </xacro:if>
+        <!-- MYNT Camera -->
+        <xacro:unless value="${camera['type'] == 'downward'}">
+          <xacro:mynt_macro
+            namespace="${namespace}"
+            name="${camera['name']}"
+            parent_link="${namespace}/origin"
+            update_rate="${camera['rate']}"
+            hfov="${camera['hfov']}"
+            width="${camera['width']}"
+            height="${camera['height']}"
+            stddev="${camera['stddev']}"
+            baseline="${camera['baseline']}">
+            <origin xyz="${camera['pose'][0]} ${camera['pose'][1]} ${camera['pose'][2]}"
+                    rpy="${camera['pose'][3]} ${camera['pose'][4]} ${camera['pose'][5]}"/>
+          </xacro:mynt_macro>
+        </xacro:unless>
       </xacro:unless>
       <xacro:cameras_macro namespace="${namespace}" cameras="${cameras[1:]}"/>

Commit message: (hopefully) fixing commit history

File: urdf/robot_sensors.xacro (robot description, xacro)
@@ -43,4 +43,29 @@
     <xacro:property name="imu" value="${config['imu']}"/>
     <xacro:imu_plugin_macro
+      namespace="${namespace}"
+      imu_suffix=""
+      parent_link="${namespace}/origin"
+      imu_topic="${imu['topic']}"
+      gyroscope_noise_density="0.0003394"
+      gyroscope_random_walk="0.000038785"
+      gyroscope_bias_correlation_time="1000.0"
+      gyroscope_turn_on_bias_sigma="0.0087"
+      accelerometer_noise_density="0.004"
+      accelerometer_random_walk="0.006"
+      accelerometer_bias_correlation_time="300.0"
+      accelerometer_turn_on_bias_sigma="0.1960"
+      orientation_noise="0.01"
+      enable_local_ned_frame="false"
+      reference_frame="${inertial_reference_frame}"
+      update_rate="${imu['rate']}">
+      <origin xyz="${imu['pose'][0]} ${imu['pose'][1]} ${imu['pose'][2]}"
+              rpy="${imu['pose'][3]} ${imu['pose'][4]} ${imu['pose'][5]}"/>
+    </xacro:imu_plugin_macro>
+  </xacro:if>
+  <!-- mynt camera has its own imu -->
+  <xacro:if value="${'mynt_imu' in config}">
+    <xacro:property name="imu" value="${config['imu']}"/>
+    <!-- TODO: I copied this over from the original macro. Fill in values for the MYNT imu. -->
+    <xacro:mynt_imu_plugin_macro
       namespace="${namespace}"
       imu_suffix=""

Commit message: Finish mynt camera/imu macro rewrite

File: urdf/robot_sensors.xacro (robot description, xacro)
@@ -65,9 +65,9 @@
   <!-- mynt camera has its own imu -->
   <xacro:if value="${'mynt_imu' in config}">
-    <xacro:property name="imu" value="${config['imu']}"/>
+    <xacro:property name="imu" value="${config['mynt_imu']}"/>
     <!-- TODO: I copied this over from the original macro. Fill in values for the MYNT imu. -->
     <xacro:mynt_imu_plugin_macro
       namespace="${namespace}"
-      imu_suffix=""
+      imu_suffix="mynt"
       parent_link="${namespace}/origin"
       imu_topic="${imu['topic']}"
@@ -86,5 +86,5 @@
       <origin xyz="${imu['pose'][0]} ${imu['pose'][1]} ${imu['pose'][2]}"
               rpy="${imu['pose'][3]} ${imu['pose'][4]} ${imu['pose'][5]}"/>
-    </xacro:imu_plugin_macro>
+    </xacro:mynt_imu_plugin_macro>
   </xacro:if>
   <!-- Pose sensor as ground truth for state estimation -->
@@ -115,5 +115,5 @@
       <!-- Downward Camera -->
       <xacro:unless value="${camera['type'] == 'stereo'}">
-        <xacro:if value="${camera['type'] == 'downward'}">
+        <xacro:if value="${camera['type'] == 'mono'}">
           <xacro:camera_macro
             namespace="${namespace}"
@@ -130,5 +130,5 @@
         </xacro:if>
         <!-- MYNT Camera -->
-        <xacro:unless value="${camera['type'] == 'downward'}">
+        <xacro:unless value="${camera['type'] == 'mono'}">
           <xacro:mynt_macro
             namespace="${namespace}"

File: urdf/snippets.xacro (robot description, xacro)
@@ -131,4 +131,53 @@
     </xacro:camera_macro>
   </xacro:macro>
+  <!-- MYNT Camera has two cameras in it; We have to handle it similarly to stereo cameras -->
+  <xacro:macro name="mynt_macro" params="namespace parent_link name update_rate hfov width height stddev baseline *origin">
+    <xacro:mynt_camera_macro
+      namespace="${namespace}"
+      name="${name}/left"
+      parent_link="${parent_link}"
+      update_rate="${update_rate}"
+      hfov="${hfov}"
+      width="${width}"
+      height="${height}"
+      stddev="${stddev}"
+      baseline="${baseline}">
+      <xacro:insert_block name="origin" />
+    </xacro:mynt_camera_macro>
+    <xacro:mynt_camera_macro
+      namespace="${namespace}"
+      name="${name}/right"
+      parent_link="${namespace}/${name}/left_link"
+      update_rate="${update_rate}"
+      hfov="${hfov}"
+      width="${width}"
+      height="${height}"
+      stddev="${stddev}"
+      baseline="${baseline}">
+      <origin xyz="0 ${-baseline} 0"/>
+    </xacro:mynt_camera_macro>
+    <!-- TODO: Add gazebo plugin support. Lots we can rip from camera_macro.
+      Would probably need to make the plugin right here so that it only runs once.
+      Uses different plugin than normal, great instructions on http://gazebosim.org/tutorials/?tut=ros_depth_camera -->
+  </xacro:macro>
+  <!-- TODO: Add camera distortion -->
+  <!-- This is the macro that actually defines one of the MYNT cameras -->
+  <xacro:macro name="mynt_camera_macro" params="namespace name parent_link update_rate hfov width height stddev baseline:=0 *origin">
+    <link name="${namespace}/${name}_link">
+        <xacro:dummy_inertia />
+        <xacro:no_collision />
+    </link>
+    <joint name="${namespace}/${name}_joint" type="fixed">
+        <xacro:insert_block name="origin" />
+        <parent link="${parent_link}" />
+        <child link="${namespace}/${name}_link" />
+    </joint>
+    <link name="${namespace}/${name}_optical" />
+    <joint name="${namespace}/${name}_optical_joint" type="fixed">
+      <parent link="${namespace}/${name}_link" />
+      <child link="${namespace}/${name}_optical" />
+      <origin rpy="${-pi/2} 0 ${-pi/2}"></origin>
+    </joint>
+  </xacro:macro>
   <xacro:macro name="dvl_single_sonar" params="namespace suffix index pitch yaw update_rate">
     <link name="${namespace}/dvl${suffix}_sonar${index}_link">
@@ -309,4 +358,29 @@
     </gazebo>
   </xacro:macro>
+  <xacro:macro name="mynt_imu_plugin_macro"
+    params="namespace imu_suffix parent_link imu_topic
+      gyroscope_noise_density gyroscope_random_walk
+      gyroscope_bias_correlation_time gyroscope_turn_on_bias_sigma
+      accelerometer_noise_density accelerometer_random_walk
+      accelerometer_bias_correlation_time accelerometer_turn_on_bias_sigma
+      orientation_noise
+      update_rate reference_frame
+      enable_local_ned_frame
+      *origin">
+    <!-- IMU link -->
+    <link name="${namespace}/imu${imu_suffix}_link">
+      <xacro:dummy_inertia/>
+    </link>
+    <!-- IMU joint -->
+    <!-- TODO: Modify this so it fits mynt imu coordinate frame @ https://mynt-eye-d-sdk.readthedocs.io/en/latest/product/imu_coord.html -->
+    <joint name="${namespace}/imu${imu_suffix}_joint" type="revolute">
+      <xacro:insert_block name="origin" />
+      <parent link="${parent_link}" />
+      <child link="${namespace}/imu${imu_suffix}_link" />
+      <limit upper="0" lower="0" effort="0" velocity="0" />
+      <axis xyz="1 0 0"/>
+    </joint>
+    <!-- TODO: implement gazebo model for the mynt imu. Probably able to copy a lot from the other imu macro. -->
+  </xacro:macro>
   <xacro:macro name="thruster_macro"
     params="namespace

Commit message: Finished mynt macro

File: urdf/robot_sensors.xacro (robot description, xacro)
@@ -63,29 +63,4 @@
     </xacro:imu_plugin_macro>
   </xacro:if>
-  <!-- mynt camera has its own imu -->
-  <xacro:if value="${'mynt_imu' in config}">
-    <xacro:property name="imu" value="${config['mynt_imu']}"/>
-    <!-- TODO: I copied this over from the original macro. Fill in values for the MYNT imu. -->
-    <xacro:mynt_imu_plugin_macro
-      namespace="${namespace}"
-      imu_suffix="_mynt"
-      parent_link="${namespace}/origin"
-      imu_topic="${imu['topic']}"
-      gyroscope_noise_density="0.0003394"
-      gyroscope_random_walk="0.000038785"
-      gyroscope_bias_correlation_time="1000.0"
-      gyroscope_turn_on_bias_sigma="0.0087"
-      accelerometer_noise_density="0.004"
-      accelerometer_random_walk="0.006"
-      accelerometer_bias_correlation_time="300.0"
-      accelerometer_turn_on_bias_sigma="0.1960"
-      orientation_noise="0.01"
-      enable_local_ned_frame="false"
-      reference_frame="${inertial_reference_frame}"
-      update_rate="${imu['rate']}">
-      <origin xyz="${imu['pose'][0]} ${imu['pose'][1]} ${imu['pose'][2]}"
-              rpy="${imu['pose'][3]} ${imu['pose'][4]} ${imu['pose'][5]}"/>
-    </xacro:mynt_imu_plugin_macro>
-  </xacro:if>
   <!-- Pose sensor as ground truth for state estimation -->
   <xacro:default_pose_3d_macro
@@ -130,7 +105,9 @@
         </xacro:if>
         <!-- MYNT Camera -->
+        <!-- Suffix isn't set here because right now we just have one, but you should just need to change the suffix for each and it'll work. -->
         <xacro:unless value="${camera['type'] == 'mono'}">
           <xacro:mynt_macro
             namespace="${namespace}"
+            mynt_suffix="${camera['suffix']}"
             name="${camera['name']}"
             parent_link="${namespace}/origin"

File: urdf/snippets.xacro (robot description, xacro)
@@ -132,10 +132,20 @@
   </xacro:macro>
   <!-- MYNT Camera has two cameras in it; We have to handle it similarly to stereo cameras -->
-  <xacro:macro name="mynt_macro" params="namespace parent_link name update_rate hfov width height stddev baseline *origin">
+  <xacro:macro name="mynt_macro" params="namespace mynt_suffix parent_link name update_rate hfov width height stddev baseline *origin">
+    <!-- Parent link is {namespace]/origin -->
+    <link name="${namespace}/${name}_${mynt_suffix}_link">
+        <xacro:dummy_inertia />
+        <xacro:no_collision />
+    </link>
+    <joint name="${namespace}/${name}_joint" type="fixed">
+        <xacro:insert_block name="origin" />
+        <parent link="${parent_link}" />
+        <child link="${namespace}/${name}_${mynt_suffix}_link" />
+    </joint>
     <!-- Left camera -->
     <xacro:mynt_camera_macro
       namespace="${namespace}"
-      name="${name}/left"
-      parent_link="${parent_link}"
+      name="${name}_${mynt_suffix}/left"
+      parent_link="${namespace}/${name}_${mynt_suffix}_link"
       update_rate="${update_rate}"
       hfov="${hfov}"
@@ -149,6 +159,6 @@
     <xacro:mynt_camera_macro
       namespace="${namespace}"
-      name="${name}/right"
-      parent_link="${namespace}/${name}/left_link"
+      name="${name}_${mynt_suffix}/right"
+      parent_link="${namespace}/${name}_${mynt_suffix}_link"
       update_rate="${update_rate}"
       hfov="${hfov}"
@@ -159,7 +169,30 @@
       <origin xyz="0 ${-baseline} 0"/>
     </xacro:mynt_camera_macro>
-    <!-- TODO: Add gazebo plugin support. Lots we can rip from camera_macro.
-      Would probably need to make the plugin right here so that it only runs once.
-      Uses different plugin than normal, great instructions on http://gazebosim.org/tutorials/?tut=ros_depth_camera -->
+    <!-- IMU needs added here rather than completely separately because its link/frame need to be relative from the camera itself -->
+    <!-- TODO: I copied these numbers over from the original macro. Fill in values for the MYNT imu. -->
+    <!-- If this macro is running, we can safely assume that this value in the .yaml exists, because if this is running we have a mynt camera initially. -->
+    <xacro:property name="imu" value="${config['mynt_imu']}"/>
+    <xacro:imu_plugin_macro
+      namespace="${namespace}"
+      imu_suffix="_mynt_${mynt_suffix}"
+      parent_link="${namespace}/${name}_${mynt_suffix}_link"
+      imu_topic="${imu['topic']}"
+      gyroscope_noise_density="0.0003394"
+      gyroscope_random_walk="0.000038785"
+      gyroscope_bias_correlation_time="1000.0"
+      gyroscope_turn_on_bias_sigma="0.0087"
+      accelerometer_noise_density="0.004"
+      accelerometer_random_walk="0.006"
+      accelerometer_bias_correlation_time="300.0"
+      accelerometer_turn_on_bias_sigma="0.1960"
+      orientation_noise="0.01"
+      enable_local_ned_frame="false"
+      reference_frame="${inertial_reference_frame}"
+      update_rate="${imu['rate']}">
+      <!-- Halfway between the two cameras -->
+      <origin xyz="0 ${-baseline/2} 0" />
+    </xacro:imu_plugin_macro>
+    <!-- TODO: Add gazebo camera plugin http://gazebosim.org/tutorials/?tut=ros_depth_camera -->
+    <!-- imu plugin is already here; We launch the mynt imu with the same macro as our original macro -->
   </xacro:macro>
   <!-- TODO: Add camera distortion -->
@@ -360,29 +393,4 @@
     </gazebo>
   </xacro:macro>
-  <xacro:macro name="mynt_imu_plugin_macro"
-    params="namespace imu_suffix parent_link imu_topic
-      gyroscope_noise_density gyroscope_random_walk
-      gyroscope_bias_correlation_time gyroscope_turn_on_bias_sigma
-      accelerometer_noise_density accelerometer_random_walk
-      accelerometer_bias_correlation_time accelerometer_turn_on_bias_sigma
-      orientation_noise
-      update_rate reference_frame
-      enable_local_ned_frame
-      *origin">
-    <!-- IMU link -->
-    <link name="${namespace}/imu${imu_suffix}_link">
-      <xacro:dummy_inertia/>
-    </link>
-    <!-- IMU joint -->
-    <!-- TODO: Modify this so it fits mynt imu coordinate frame @ https://mynt-eye-d-sdk.readthedocs.io/en/latest/product/imu_coord.html -->
-    <joint name="${namespace}/imu${imu_suffix}_joint" type="revolute">
-      <xacro:insert_block name="origin" />
-      <parent link="${parent_link}" />
-      <child link="${namespace}/imu${imu_suffix}_link" />
-      <limit upper="0" lower="0" effort="0" velocity="0" />
-      <axis xyz="1 0 0"/>
-    </joint>
-    <!-- TODO: implement gazebo model for the mynt imu. Probably able to copy a lot from the other imu macro. -->
-  </xacro:macro>
   <xacro:macro name="thruster_macro"
     params="namespace

Commit message: Redid/reorganized mynt namespacing, modified mynt imu handling

File: urdf/robot_sensors.xacro (robot description, xacro)
@@ -109,5 +109,4 @@
           <xacro:mynt_macro
             namespace="${namespace}"
-            mynt_suffix="${camera['suffix']}"
             name="${camera['name']}"
             parent_link="${namespace}/origin"
@@ -117,5 +116,7 @@
             height="${camera['height']}"
             stddev="${camera['stddev']}"
-            baseline="${camera['baseline']}">
+            baseline="${camera['baseline']}"
+            imu_topic="${camera['imu_topic']}"
+            imu_rate="${camera['imu_rate']}">
             <origin xyz="${camera['pose'][0]} ${camera['pose'][1]} ${camera['pose'][2]}"
                     rpy="${camera['pose'][3]} ${camera['pose'][4]} ${camera['pose'][5]}"/>

File: urdf/snippets.xacro (robot description, xacro)
@@ -132,7 +132,7 @@
   </xacro:macro>
   <!-- MYNT Camera has two cameras in it; We have to handle it similarly to stereo cameras -->
-  <xacro:macro name="mynt_macro" params="namespace mynt_suffix parent_link name update_rate hfov width height stddev baseline *origin">
+  <xacro:macro name="mynt_macro" params="namespace parent_link name update_rate hfov width height stddev baseline imu_topic imu_rate *origin">
     <!-- Parent link is {namespace]/origin -->
-    <link name="${namespace}/${name}_${mynt_suffix}_link">
+    <link name="${namespace}/${name}/base_link">
         <xacro:dummy_inertia />
         <xacro:no_collision />
@@ -141,11 +141,11 @@
         <xacro:insert_block name="origin" />
         <parent link="${parent_link}" />
-        <child link="${namespace}/${name}_${mynt_suffix}_link" />
+        <child link="${namespace}/${name}/base_link" />
     </joint>
     <!-- Left camera -->
     <xacro:mynt_camera_macro
       namespace="${namespace}"
-      name="${name}_${mynt_suffix}/left"
-      parent_link="${namespace}/${name}_${mynt_suffix}_link"
+      name="${name}/left"
+      parent_link="${namespace}/${name}/base_link"
       update_rate="${update_rate}"
       hfov="${hfov}"
@@ -159,6 +159,6 @@
     <xacro:mynt_camera_macro
       namespace="${namespace}"
-      name="${name}_${mynt_suffix}/right"
-      parent_link="${namespace}/${name}_${mynt_suffix}_link"
+      name="${name}/right"
+      parent_link="${namespace}/${name}/base_link"
       update_rate="${update_rate}"
       hfov="${hfov}"
@@ -172,10 +172,9 @@
     <!-- TODO: I copied these numbers over from the original macro. Fill in values for the MYNT imu. -->
     <!-- If this macro is running, we can safely assume that this value in the .yaml exists, because if this is running we have a mynt camera initially. -->
-    <xacro:property name="imu" value="${config['mynt_imu']}"/>
     <xacro:imu_plugin_macro
-      namespace="${namespace}"
-      imu_suffix="_mynt_${mynt_suffix}"
-      parent_link="${namespace}/${name}_${mynt_suffix}_link"
-      imu_topic="${imu['topic']}"
+      namespace="${namespace}/${name}"
+      imu_suffix=""
+      parent_link="${namespace}/${name}/base_link"
+      imu_topic="${imu_topic}"
       gyroscope_noise_density="0.0003394"
       gyroscope_random_walk="0.000038785"
@@ -189,5 +188,5 @@
       enable_local_ned_frame="false"
       reference_frame="${inertial_reference_frame}"
-      update_rate="${imu['rate']}">
+      update_rate="${imu_rate}">
       <!-- Halfway between the two cameras -->
       <origin xyz="0 ${-baseline/2} 0" />

Commit message: various tweaks

File: urdf/robot_sensors.xacro (robot description, xacro)
@@ -3,46 +3,40 @@
   <!-- Everything here is ENU frame -->
   <!-- DVL  -->
-  <!-- TODO: restore below if when xacro releases 1.14.4 -->
-  <!-- <xacro:if value="${'dvl' in config}"> -->
-    <xacro:property name="dvl" value="${config['dvl']}"/>
-    <xacro:dvl_plugin_macro
-      namespace="${namespace}"
-      suffix=""
-      parent_link="${namespace}/origin"
-      topic="${dvl['topic']}"
-      scale="1"
-      update_rate="${dvl['rate']}"
-      reference_frame="${inertial_reference_frame}"
-      noise_sigma="${dvl['sigma']}"
-      noise_amplitude="1">
-      <origin xyz="${dvl['pose'][0]} ${dvl['pose'][1]} ${dvl['pose'][2]}"
-              rpy="${dvl['pose'][3]} ${dvl['pose'][4]} ${dvl['pose'][5]}"/>
-    </xacro:dvl_plugin_macro>
-  <!-- </xacro:if> -->
+  <!--datasheet: nortekgroup.com/products/dvl-1000-300m/pdf -->
+  <xacro:property name="dvl" value="${config['dvl']}"/>
+  <xacro:dvl_plugin_macro
+    namespace="${namespace}"
+    suffix=""
+    parent_link="${namespace}/origin"
+    topic="${dvl['topic']}"
+    scale="1"
+    update_rate="${dvl['rate']}"
+    reference_frame="${inertial_reference_frame}"
+    noise_sigma="${dvl['sigma']}"
+    noise_amplitude="1">
+    <origin xyz="${dvl['pose'][0]} ${dvl['pose'][1]} ${dvl['pose'][2]}"
+            rpy="${dvl['pose'][3]} ${dvl['pose'][4]} ${dvl['pose'][5]}"/>
+  </xacro:dvl_plugin_macro>
   <!-- Pressure  -->
-  <!-- TODO: restore below if when xacro releases 1.14.4 -->
-  <!-- <xacro:if value="${'depth' in config}"> -->
-    <xacro:property name="depth" value="${config['depth']}"/>
-    <xacro:pressure_plugin_macro
-      namespace="${namespace}"
-      suffix=""
-      parent_link="${namespace}/origin"
-      topic="${depth['topic']}"
-      update_rate="${depth['rate']}"
-      range="300"
-      noise_sigma="${depth['sigma'] * 9.80638}"
-      noise_amplitude="1"
-      estimateDepth="false"
-      standardPressure="101.325"
-      kPaPerM="9.80638">
-      <origin xyz="${depth['pose'][0]} ${depth['pose'][1]} ${depth['pose'][2]}"
-              rpy="${depth['pose'][3]} ${depth['pose'][4]} ${depth['pose'][5]}"/>
-    </xacro:pressure_plugin_macro>
-  <!-- </xacro:if> -->
+  <xacro:property name="depth" value="${config['depth']}"/>
+  <xacro:pressure_plugin_macro
+    namespace="${namespace}"
+    suffix=""
+    parent_link="${namespace}/origin"
+    topic="${depth['topic']}"
+    update_rate="${depth['rate']}"
+    range="300"
+    noise_sigma="${depth['sigma'] * 9.80638}"
+    noise_amplitude="1"
+    estimateDepth="false"
+    standardPressure="101.325"
+    kPaPerM="9.80638">
+    <origin xyz="${depth['pose'][0]} ${depth['pose'][1]} ${depth['pose'][2]}"
+            rpy="${depth['pose'][3]} ${depth['pose'][4]} ${depth['pose'][5]}"/>
+  </xacro:pressure_plugin_macro>
   <!-- IMU  -->
-  <!-- TODO: Get imu model from config -->
-  <!-- TODO: restore below if when xacro releases 1.14.4 -->
-  <!-- <xacro:if value="${'imu' in config}"> -->
-    <xacro:property name="imu" value="${config['imu']}"/>
+  <!-- datasheet: microstrain.com/sites/default/files/3dm0gx4-25_datasheet_8400-0060.pdf -->
+  <!-- TODO: orientation noise to be experimentally obtained -->
+    <xacro:property name="microstrain_imu" value="${config['imu']}"/>
     <xacro:imu_plugin_macro
       namespace="${namespace}"
@@ -65,5 +59,4 @@
               rpy="${imu['pose'][3]} ${imu['pose'][4]} ${imu['pose'][5]}"/>
     </xacro:imu_plugin_macro>
-  <!-- </xacro:if> -->
   <!-- Pose sensor as ground truth for state estimation -->
   <xacro:default_pose_3d_macro
