Commit message: add / fix plugins

File: urdf/robot_sensors.xacro (robot description, xacro)
@@ -2,4 +2,9 @@
 <robot xmlns:xacro="http://www.ros.org/wiki/xacro" >
   <!-- Everything here is ENU frame -->
+  <xacro:property name="dvl" value="${config['dvl']}"/>
+  <xacro:default_joint_state_publisher
+  namespace="${namespace}"
+  update_rate="${dvl['rate']}" >
+  </xacro:default_joint_state_publisher>
   <!-- DVL  -->
   <!-- TODO: restore below if when xacro releases 1.14.4 -->

File: urdf/snippets.xacro (robot description, xacro)
@@ -30,5 +30,7 @@
         <gazebo>
             <plugin name="pose_3d_plugin" filename="libuuv_gazebo_ros_pose_gt_plugin.so">
-                <robot_namespace>${namespace}</robot_namespace>
+                <ros>
+                    <namespace>${namespace}</namespace> <!-- (string, required): ros namespace in which the messages are published -->
+                </ros>
                 <link_name>${namespace}/base_link</link_name>
                 <sensor_topic>pose_gt</sensor_topic>
@@ -171,4 +173,7 @@
                 </ray>
                 <plugin filename="libgazebo_ros_ray_sensor.so" name="dvl${suffix}_sonar${index}">
+                    <ros>
+                        <namespace>${namespace}</namespace>
+                    </ros>
                     <gaussianNoise>0.005</gaussianNoise>
                     <alwaysOn>true</alwaysOn>
@@ -202,5 +207,7 @@
         <gazebo>
             <plugin filename="libuuv_gazebo_ros_dvl_plugin.so" name="libuuv_gazebo_dvl${suffix}_plugin">
-                <robot_namespace>${namespace}</robot_namespace> <!-- (string, required): ros namespace in which the messages are published -->
+                <ros>
+                    <namespace>${namespace}</namespace>
+                </ros> <!-- (string, required): ros namespace in which the messages are published -->
                 <link_name>${namespace}/dvl${suffix}_link</link_name>
                 <sensor_topic>${topic}</sensor_topic> <!-- (string): name of the sensor output topic and prefix of service names -->
@@ -344,3 +351,14 @@
         </gazebo>
     </xacro:macro>
+    <xacro:macro name="default_joint_state_publisher" params="namespace update_rate">
+        <gazebo>
+            <plugin name="uuv_joint_state_publisher" filename="libuuv_joint_state_publisher.so">
+                <ros>
+                    <namespace>${namespace}</namespace>
+                </ros>
+                <!-- <robotNamespace>${namespace}</robotNamespace> -->
+                <updateRate>${update_rate}</updateRate>
+            </plugin>
+        </gazebo>
+    </xacro:macro>
 </robot>

Commit message: Link to ZED camera

File: urdf/robot_sensors.xacro (robot description, xacro)
@@ -112,8 +112,12 @@
           </xacro:camera_macro>
         </xacro:if>
-        <!-- MYNT Camera -->
+        <!-- MYNT/ZED Camera -->
         <!-- Suffix isn't set here because right now we just have one, but you should just need to change the suffix for each and it'll work. -->
         <xacro:unless value="${camera['type'] == 'mono'}">
-          <xacro:mynt_macro
+          <!-- <xacro:include filename="$(find zed_wrapper)/urdf/zed_macro.urdf.xacro" /> -->
+          <!-- <xacro:zed_camera name="${camera['name']}" model="${camera['model']}" parent="${namespace}/base_link" >
+            <origin xyz="${camera['pose'][0]} ${camera['pose'][1]} ${camera['pose'][2]}" rpy="${camera['pose'][3]} ${camera['pose'][4]} ${camera['pose'][5]}" />
+          </xacro:zed_camera> -->
+          <!-- <xacro:mynt_macro
             namespace="${namespace}"
             name="${camera['name']}"
@@ -129,5 +133,5 @@
             <origin xyz="${camera['pose'][0]} ${camera['pose'][1]} ${camera['pose'][2]}"
                     rpy="${camera['pose'][3]} ${camera['pose'][4]} ${camera['pose'][5]}"/>
-          </xacro:mynt_macro>
+          </xacro:mynt_macro> -->
         </xacro:unless>
       </xacro:unless>

Commit message: got stereo camera working in tf

File: urdf/robot_sensors.xacro (robot description, xacro)
@@ -54,5 +54,6 @@
           namespace="${namespace}"
           parent_link="${namespace}/origin"
-          name="${camera['name']}">
+          name="${camera['name']}"
+          baseline="${camera['baseline']}">
           <origin xyz="${camera['pose'][0]} ${camera['pose'][1]} ${camera['pose'][2]}"
                   rpy="${camera['pose'][3]} ${camera['pose'][4]} ${camera['pose'][5]}"/>

File: urdf/snippets.xacro (robot description, xacro)
@@ -45,4 +45,21 @@
             <origin rpy="${-pi/2} 0 ${-pi/2}"></origin>
         </joint>
+    </xacro:macro>
+    <xacro:macro name="stereo_macro" params="namespace parent_link name baseline *origin">
+        <link name="${namespace}/stereo_link">
+            <xacro:dummy_inertia />
+            <xacro:no_collision />
+        </link>
+        <joint name="${namespace}/stereo_joint" type="fixed">
+            <xacro:insert_block name="origin" />
+            <parent link="${parent_link}" />
+            <child link="${namespace}/stereo_link" />
+        </joint>
+        <xacro:camera_macro namespace="${namespace}/${name}" name="left" parent_link="${namespace}/stereo_link">
+            <origin xyz="0 0 0" />
+        </xacro:camera_macro>
+        <xacro:camera_macro namespace="${namespace}/${name}" name="right" parent_link="${namespace}/stereo_link">
+            <origin xyz="0 ${-baseline} 0" />
+        </xacro:camera_macro>
     </xacro:macro>
     <xacro:macro name="dvl_plugin_macro" params="namespace suffix parent_link *origin">
