Commit message: Ubuntu 16 cmpatibility and removing uuv dependency

File: urdf/robot_actuators.xacro (robot description, xacro)
@@ -15,5 +15,5 @@
   <!-- Macro makes any number of thrusters from config -->
   <xacro:macro name="thrusters_macro" params="namespace config thrusters index">
-    <xacro:if value="${len(thrusters)}">
+    <xacro:if value="${thrusters != []}">
       <xacro:property name="thruster" value="${thrusters[0]}"/>
       <xacro:thruster_macro

File: urdf/robot_base.xacro (robot description, xacro)
@@ -2,9 +2,6 @@
 <!-- All coordinates in file must follow ROS conventions: x forward, z up -->
 <robot xmlns:xacro="http://www.ros.org/wiki/xacro" >
-  <xacro:include filename="$(find uuv_descriptions)/urdf/common.urdf.xacro"/>
-  <xacro:include filename="$(find uuv_sensor_ros_plugins)/urdf/sensor_snippets.xacro"/>
   <xacro:include filename="$(find riptide_descriptions)/urdf/snippets.xacro" />
   <xacro:include filename="$(find riptide_descriptions)/urdf/robot.gazebo.xacro" />
-  <xacro:include filename="$(find uuv_gazebo_ros_plugins)/urdf/snippets.xacro"/>
   <xacro:macro name="robot_base"
     params="namespace config inertial_reference_frame">

File: urdf/robot_sensors.xacro (robot description, xacro)
@@ -70,5 +70,5 @@
   <!-- Builds any number of cameras from yaml -->
   <xacro:macro name="cameras_macro" params="namespace cameras">
-    <xacro:if value="${len(cameras)}">
+    <xacro:if value="${cameras != []}">
       <xacro:property name="camera" value="${cameras[0]}"/>
       <xacro:if value="${camera['type'] == 'stereo'}">

File: urdf/snippets.xacro (robot description, xacro)
@@ -7,4 +7,38 @@
       <inertia ixx="0" ixy="0.0" ixz="0.0" iyy="0" iyz="0.0" izz="0" />
     </inertial>
+  </xacro:macro>
+  <xacro:macro name="no_collision">
+    <collision>
+      <geometry>
+        <cylinder length="${0.000001}" radius="${0.000001}" />
+      </geometry>
+      <origin xyz="0 0 0" rpy="0 ${0.5*pi} 0"/>
+    </collision>
+  </xacro:macro>
+  <!-- Ground truth position -->
+  <xacro:macro name="default_pose_3d_macro" params="namespace parent_link inertial_reference_frame">
+    <!-- Mount a 3D pose sensor -->
+    <link name="${namespace}/pose_sensor_link">
+      <xacro:dummy_inertia />
+    </link>
+    <joint name="${namespace}/pose_sensor_joint" type="revolute">
+      <axis xyz="0 0 1"/>
+      <parent link="${parent_link}"/>
+      <child link="${namespace}/pose_sensor_link"/>
+      <limit effort="0" lower="0" upper="0" velocity="0"/>
+    </joint>
+    <gazebo>
+      <plugin name="pose_3d_plugin" filename="libuuv_gazebo_ros_pose_gt_plugin.so">
+        <robot_namespace>${namespace}</robot_namespace>
+        <link_name>${namespace}/base_link</link_name>
+        <sensor_topic>pose_gt</sensor_topic>
+        <static_reference_frame>${inertial_reference_frame}</static_reference_frame>
+        <noise_sigma>0</noise_sigma>
+        <noise_amplitude>0</noise_amplitude>
+        <update_rate>20</update_rate>
+        <enable_gazebo_messages>false</enable_gazebo_messages>
+        <publish_ned_odom>false</publish_ned_odom>
+      </plugin>
+    </gazebo>
   </xacro:macro>
   <!-- TODO: Add camera distortion -->

Commit message: Starting claw

File: urdf/robot_actuators.xacro (robot description, xacro)
@@ -32,4 +32,13 @@
     </xacro:if>
   </xacro:macro>
+  <xacro:if value="${'claw' in config}">
+    <xacro:property name="claw" value="${config['claw']}"/>
+    <xacro:newton_gripper_macro
+      namespace="${namespace}"
+      parent_link="${namespace}/origin">
+      <origin xyz="${claw['pose'][0]} ${claw['pose'][1]} ${claw['pose'][2]}"
+              rpy="${claw['pose'][3]} ${claw['pose'][4]} ${claw['pose'][5]}"/>
+    </xacro:newton_gripper_macro>
+  </xacro:if>
   <xacro:thrusters_macro
         namespace="${namespace}"

File: urdf/snippets.xacro (robot description, xacro)
@@ -348,3 +348,64 @@
     </gazebo>
   </xacro:macro>
+  <xacro:macro name="newton_gripper_macro" params="namespace parent_link *origin">
+    <link name="${namespace}/gripper_base_link">
+      <xacro:dummy_inertia />
+    </link>
+    <joint name="${namespace}/gripper_base_joint" type="fixed">
+      <parent link="${parent_link}"/>
+      <child link="${namespace}/gripper_base_link"/>
+      <xacro:insert_block name="origin" />
+    </joint>
+    <link name="${namespace}/gripper_inner_link">
+      <inertial>
+        <mass value="0.00001" />
+        <inertia ixx="0.001" ixy="0.0" ixz="0.0" iyy="0.001" iyz="0.0" izz="0.001" />
+      </inertial>
+      <visual>
+        <geometry>
+          <mesh filename="package://riptide_descriptions/meshes/claw_inside.dae" scale="0.0254 0.0254 0.0254"/>
+        </geometry>
+        <origin xyz="0 0 0" rpy="0 ${0.5*pi} 0"/>
+      </visual>
+      <collision>
+        <geometry>
+          <mesh filename="package://riptide_descriptions/meshes/claw_inside.dae" scale="0.0254 0.0254 0.0254"/>
+        </geometry>
+        <origin xyz="0 0 0" rpy="0 ${0.5*pi} 0"/>
+      </collision>
+    </link>
+    <joint name="${namespace}/gripper_inner_joint" type="revolute">
+      <axis xyz="0 0 1"/>
+      <parent link="${namespace}/gripper_base_link"/>
+      <child link="${namespace}/gripper_inner_link"/>
+      <origin xyz="-0.032 0.02 0" />
+      <limit effort="100" lower="0" upper="0.52" velocity=".32"/>
+    </joint>
+    <link name="${namespace}/gripper_outer_link">
+      <inertial>
+        <mass value="0.00001" />
+        <inertia ixx="0.001" ixy="0.0" ixz="0.0" iyy="0.001" iyz="0.0" izz="0.001" />
+      </inertial>
+      <visual>
+        <geometry>
+          <mesh filename="package://riptide_descriptions/meshes/claw_outside.dae" scale="0.0254 0.0254 0.0254"/>
+        </geometry>
+        <origin xyz="0 0 0" rpy="0 ${0.5*pi} 0"/>
+      </visual>
+      <collision>
+        <geometry>
+          <mesh filename="package://riptide_descriptions/meshes/claw_outside.dae" scale="0.0254 0.0254 0.0254"/>
+        </geometry>
+        <origin xyz="0 0 0" rpy="0 ${0.5*pi} 0"/>
+      </collision>
+    </link>
+    <joint name="${namespace}/gripper_outer_joint" type="revolute">
+      <axis xyz="0 0 1"/>
+      <parent link="${namespace}/gripper_base_link"/>
+      <child link="${namespace}/gripper_outer_link"/>
+      <origin xyz="-0.032 -0.02 0" />
+      <limit effort="100" lower="-0.52" upper="0" velocity=".32"/>
+      <mimic joint="${namespace}/gripper_inner_joint" multiplier="-1" />
+    </joint>
+  </xacro:macro>
 </robot>

Commit message: added actuator macros with simple boxes for sim

File: urdf/robot_actuators.xacro (robot description, xacro)
@@ -31,4 +31,40 @@
     </xacro:if>
   </xacro:macro>
+  <xacro:macro name="claw_macro" params="namespace config">
+    <xacro:property name="claw" value="config['claw']"/>
+    <joint name="${namespace}/claw_joint" type="fixed">
+      <origin xyz="${claw['pose'][0]} ${claw['pose'][1]} ${claw['pose'][2]}"
+              rpy="${claw['pose'][3]} ${claw['pose'][4]} ${claw['pose'][5]}"/>
+      <parent link="${namespace}/origin"/>
+      <child link="${namespace}/claw_link"/>
+    </joint>
+    <link name="${namespace}/claw_link">
+      <xacro:dummy_inertia />
+      <xacro:no_collision />
+      <visual>
+        <geometry>
+          <box size="0.1 0.025 0.025"/>
+        </geometry>
+      </visual>
+    </link>
+  </xacro:macro>
+  <xacro:macro name="torpedo_macro" params="namespace config">
+    <xacro:property name="torpedos" value="config['torpedos']"/>
+    <joint name="${namespace}/torpedo_joint" type="fixed">
+      <origin xyz="${torpedo['pose'][0]} ${torpedo['pose'][1]} ${torpedo['pose'][2]}"
+              rpy="${torpedo['pose'][3]} ${torpedo['pose'][4]} ${torpedo['pose'][5]}" />
+      <parent link="${namespace}/origin"/>
+      <child link="${namespace}/claw_link"/>
+    </joint>
+    <link name="${namespace}/torpedo_link">
+      <xacro:dummy_inertia />
+      <xacro:no_collision />
+      <visual>
+        <geometry>
+          <box size="0.1 0.025 0.025"/>
+        </geometry>
+      </visual>
+    </link>
+  </xacro:macro>
   <xacro:thrusters_macro
         namespace="${namespace}"
@@ -36,3 +72,9 @@
         thrusters="${config['thrusters']}"
         index="0"/>
+  <xacro:claw_macro
+        namespace="${namespace}"
+        config="${config}"/>
+  <xacro:torpedo_macro
+        namespace="${namespace}"
+        config="${config}"/>
 </robot>

Commit message: added marker droppers

File: urdf/robot_actuators.xacro (robot description, xacro)
@@ -20,5 +20,6 @@
         namespace="${namespace}"
         thruster_id="${index}"
-        mesh_filename="${prop_file}">
+        mesh_filename="${config['mesh']}"
+        rotor_constant="${config['rotor_constant']}">
         <origin xyz="${thruster['pose'][0]} ${thruster['pose'][1]} ${thruster['pose'][2]}"
                 rpy="${thruster['pose'][3]} ${thruster['pose'][4]} ${thruster['pose'][5]}"/>
@@ -32,5 +33,5 @@
   </xacro:macro>
   <xacro:macro name="claw_macro" params="namespace config">
-    <xacro:property name="claw" value="config['claw']"/>
+    <xacro:property name="claw" value="${config['claw']}"/>
     <joint name="${namespace}/claw_joint" type="fixed">
       <origin xyz="${claw['pose'][0]} ${claw['pose'][1]} ${claw['pose'][2]}"
@@ -44,5 +45,5 @@
       <visual>
         <geometry>
-          <box size="0.1 0.025 0.025"/>
+          <box size="0.2 0.05 0.05"/>
         </geometry>
       </visual>
@@ -50,10 +51,10 @@
   </xacro:macro>
   <xacro:macro name="torpedo_macro" params="namespace config">
-    <xacro:property name="torpedos" value="config['torpedos']"/>
+    <xacro:property name="torpedo" value="${config['torpedos']}"/>
     <joint name="${namespace}/torpedo_joint" type="fixed">
       <origin xyz="${torpedo['pose'][0]} ${torpedo['pose'][1]} ${torpedo['pose'][2]}"
               rpy="${torpedo['pose'][3]} ${torpedo['pose'][4]} ${torpedo['pose'][5]}" />
       <parent link="${namespace}/origin"/>
-      <child link="${namespace}/claw_link"/>
+      <child link="${namespace}/torpedo_link"/>
     </joint>
     <link name="${namespace}/torpedo_link">
@@ -62,5 +63,23 @@
       <visual>
         <geometry>
-          <box size="0.1 0.025 0.025"/>
+          <box size="0.25 0.05, 0.05"/>
+        </geometry>
+      </visual>
+    </link>
+  </xacro:macro>
+  <xacro:macro name="dropper_macro" params="namespace config">
+    <xacro:property name="dropper" value="${config['droppers']}"/>
+    <joint name="${namespace}/dropper_joint" type="fixed">
+      <origin xyz="${dropper['pose'][0]} ${dropper['pose'][1]} ${dropper['pose'][2]}"
+              rpy="${dropper['pose'][3]} ${dropper['pose'][4]} ${dropper['pose'][5]}" />
+      <parent link="${namespace}/origin"/>
+      <child link="${namespace}/droppers_link"/>
+    </joint>
+    <link name="${namespace}/droppers_link">
+      <xacro:dummy_inertia />
+      <xacro:no_collision />
+      <visual>
+        <geometry>
+          <box size="0.025 0.025 0.1"/>
         </geometry>
       </visual>
@@ -78,3 +97,6 @@
         namespace="${namespace}"
         config="${config}"/>
+  <xacro:dropper_macro
+        namespace="${namespace}"
+        config="${config}"/>
 </robot>

Commit message: wokring stereo and torpedo macro

File: urdf/robot_actuators.xacro (robot description, xacro)
@@ -62,5 +62,5 @@
       <visual>
         <geometry>
-          <box size="0.25 0.05, 0.05"/>
+          <box size="0.25 0.05 0.05"/>
         </geometry>
       </visual>

File: urdf/snippets.xacro (robot description, xacro)
@@ -47,17 +47,8 @@
     </xacro:macro>
     <xacro:macro name="stereo_macro" params="namespace parent_link name baseline *origin">
-        <link name="${namespace}/stereo_link">
-            <xacro:dummy_inertia />
-            <xacro:no_collision />
-        </link>
-        <joint name="${namespace}/stereo_joint" type="fixed">
+        <xacro:camera_macro namespace="${namespace}/${name}" name="left" parent_link="${namespace}/origin">
             <xacro:insert_block name="origin" />
-            <parent link="${parent_link}" />
-            <child link="${namespace}/stereo_link" />
-        </joint>
-        <xacro:camera_macro namespace="${namespace}/${name}" name="left" parent_link="${namespace}/stereo_link">
-            <origin xyz="0 0 0" />
         </xacro:camera_macro>
-        <xacro:camera_macro namespace="${namespace}/${name}" name="right" parent_link="${namespace}/stereo_link">
+        <xacro:camera_macro namespace="${namespace}/${name}" name="right" parent_link="${namespace}/${name}/left_link">
             <origin xyz="0 ${-baseline} 0" />
         </xacro:camera_macro>
